File: output/pcbs/tutorial.kicad_pcb (KiCad board)
At the start: 2 copper layers, 399 x 122.7 mm, 0 parts

Commit message: pcb shifted
Other:
- board size 399 x 122.7 mm -> 384.2 x 120.8 mm
Changed lines of the file:
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@@
     (add_net "")
   )
-            (gr_line (start 88.5 109.5) (end 88.5 -4.5) (angle 90) (layer Edge.Cuts) (width 0.15))
-(gr_line (start 90.5 -6.5) (end 480.3714400030863 -6.5) (angle 90) (layer Edge.Cuts) (width 0.15))
-(gr_line (start 482.3656720030863 -4.651785799999743) (end 487.4471405147384 62.110910785262604) (angle 90) (layer Edge.Cuts) (width 0.15))
-(gr_line (start 486.86712211473804 63.67691018526199) (end 458.0261645520557 92.51786774794425) (angle 90) (layer Edge.Cuts) (width 0.15))
-(gr_line (start 457.5596411745086 92.86487058967151) (end 414.61686575110554 115.97188426994268) (angle 90) (layer Edge.Cuts) (width 0.15))
-(gr_line (start 413.4629485286526 116.20000702821548) (end 368.2278378891291 111.51066079999998) (angle 90) (layer Edge.Cuts) (width 0.15))
-(gr_line (start 368.0216108891291 111.5) (end 90.5 111.5) (angle 90) (layer Edge.Cuts) (width 0.15))
-(gr_arc (start 90.5 -4.5) (end 90.5 -6.5) (angle -90) (layer Edge.Cuts) (width 0.15))
-(gr_arc (start 480.3714400030863 -4.5) (end 482.36567200308633 -4.6517858) (angle -85.64747217200396) (layer Edge.Cuts) (width 0.15))
-(gr_arc (start 485.4529085147384 62.26269658526235) (end 486.8671221147384 63.676910185262344) (angle -49.352527827995914) (layer Edge.Cuts) (width 0.15))
-(gr_arc (start 456.61195095205574 91.10365414794433) (end 457.55964115205575 92.86487054794432) (angle -16.71581849354868) (layer Edge.Cuts) (width 0.15))
-(gr_arc (start 413.66917552865266 114.21066782821546) (end 413.46294852865265 116.20000702821547) (angle -34.20266956466713) (layer Edge.Cuts) (width 0.15))
-(gr_arc (start 368.0216108891291 113.5) (end 368.2278378891291 111.5106608) (angle -5.918488058213384) (layer Edge.Cuts) (width 0.15))
-(gr_arc (start 90.5 109.5) (end 88.5 109.5) (angle -90) (layer Edge.Cuts) (width 0.15))
+            (gr_line (start 18.5 209.5) (end 18.5 95.5) (angle 90) (layer Edge.Cuts) (width 0.15))
+(gr_line (start 20.5 93.5) (end 400.6645391752075 93.5) (angle 90) (layer Edge.Cuts) (width 0.15))
+(gr_line (start 402.6642303769645 95.5351464000305) (end 401.5019988245296 161.66140547725809) (angle 90) (layer Edge.Cuts) (width 0.15))
+(gr_line (start 400.9165212227726 163.0404726772274) (end 371.9956889763156 191.96130492368434) (angle 90) (layer Edge.Cuts) (width 0.15))
+(gr_line (start 371.532574334482 192.30646924629917) (end 331.24907763504154 214.08325460740116) (angle 90) (layer Edge.Cuts) (width 0.15))
+(gr_line (start 330.16262507641704 214.31929129153855) (end 288.6675988965592 211.50458539324782) (angle 90) (layer Edge.Cuts) (width 0.15))
+(gr_line (start 288.53224529610117 211.5) (end 20.5 211.5) (angle 90) (layer Edge.Cuts) (width 0.15))
+(gr_arc (start 20.5 95.5) (end 20.5 93.5) (angle -90) (layer Edge.Cuts) (width 0.15))
+(gr_arc (start 400.6645391752075 95.5) (end 402.66423037520747 95.5351464) (angle -91.00692200215337) (layer Edge.Cuts) (width 0.15))
+(gr_arc (start 399.5023076227726 161.6262590772276) (end 400.9165212227726 163.0404726772276) (angle -43.99307799784316) (layer Edge.Cuts) (width 0.15))
+(gr_arc (start 370.58147537631555 190.5470913236844) (end 371.53257437631555 192.30646922368442) (angle -16.604867038568216) (layer Edge.Cuts) (width 0.15))
+(gr_arc (start 330.2979786768751 212.3238766847864) (end 330.16262507687514 214.3192912847864) (angle -32.27569407266526) (layer Edge.Cuts) (width 0.15))
+(gr_arc (start 288.53224529610117 213.5) (end 288.66759889610114 211.5045854) (angle -3.8805611112295253) (layer Edge.Cuts) (width 0.15))
+(gr_arc (start 20.5 209.5) (end 18.5 209.5) (angle -90) (layer Edge.Cuts) (width 0.15))
 )

Commit message: pcb with pro micro
Parts:
- added D1: , ComboDiode, F.Cu at (25.0, 155.0)
- added D10: , ComboDiode, F.Cu at (53.5, 98.0)
- added D11: , ComboDiode, F.Cu at (44.0, 79.0)
- added D12: , ComboDiode, F.Cu at (63.0, 155.0)
- added D13: , ComboDiode, F.Cu at (72.5, 136.0)
- added D14: , ComboDiode, F.Cu at (72.5, 117.0)
- added D15: , ComboDiode, F.Cu at (72.5, 98.0)
- added D16: , ComboDiode, F.Cu at (63.0, 79.0)
- added D17: , ComboDiode, F.Cu at (63.0, 60.0)
- added D18: , ComboDiode, F.Cu at (82.0, 155.0)
- added D19: , ComboDiode, F.Cu at (91.5, 136.0)
- added D2: , ComboDiode, F.Cu at (25.0, 136.0)
- added D20: , ComboDiode, F.Cu at (91.5, 117.0)
- added D21: , ComboDiode, F.Cu at (91.5, 98.0)
- added D22: , ComboDiode, F.Cu at (82.0, 79.0)
- added D23: , ComboDiode, F.Cu at (82.0, 60.0)
- added D24: , ComboDiode, F.Cu at (120.0, 155.0)
- added D25: , ComboDiode, F.Cu at (110.5, 136.0)
- added D26: , ComboDiode, F.Cu at (110.5, 117.0)
- added D27: , ComboDiode, F.Cu at (110.5, 98.0)
- added D28: , ComboDiode, F.Cu at (101.0, 79.0)
- added D29: , ComboDiode, F.Cu at (101.0, 60.0)
- added D3: , ComboDiode, F.Cu at (25.0, 117.0)
- added D30: , ComboDiode, F.Cu at (129.5, 136.0)
- added D31: , ComboDiode, F.Cu at (129.5, 117.0)
- added D32: , ComboDiode, F.Cu at (129.5, 98.0)
- added D33: , ComboDiode, F.Cu at (120.0, 79.0)
- added D34: , ComboDiode, F.Cu at (120.0, 60.0)
- added D35: , ComboDiode, F.Cu at (181.9, 155.0)
- added D36: , ComboDiode, F.Cu at (172.4, 136.0)
- added D37: , ComboDiode, F.Cu at (172.4, 117.0)
- added D38: , ComboDiode, F.Cu at (172.4, 98.0)
- added D39: , ComboDiode, F.Cu at (172.4, 79.0)
- added D4: , ComboDiode, F.Cu at (25.0, 98.0)
- added D40: , ComboDiode, F.Cu at (162.9, 60.0)
- added D41: , ComboDiode, F.Cu at (191.4, 136.0)
- added D42: , ComboDiode, F.Cu at (191.4, 117.0)
- added D43: , ComboDiode, F.Cu at (191.4, 98.0)
- added D44: , ComboDiode, F.Cu at (191.4, 79.0)
- added D45: , ComboDiode, F.Cu at (181.9, 60.0)
- added D46: , ComboDiode, F.Cu at (210.4, 136.0)
- added D47: , ComboDiode, F.Cu at (210.4, 117.0)
- added D48: , ComboDiode, F.Cu at (210.4, 98.0)
- added D49: , ComboDiode, F.Cu at (210.4, 79.0)
- added D5: , ComboDiode, F.Cu at (25.0, 79.0)
- added D50: , ComboDiode, F.Cu at (200.9, 60.0)
- added D51: , ComboDiode, F.Cu at (219.9, 155.0)
- added D52: , ComboDiode, F.Cu at (229.4, 136.0)
- added D53: , ComboDiode, F.Cu at (229.4, 117.0)
- added D54: , ComboDiode, F.Cu at (229.4, 98.0)
- added D55: , ComboDiode, F.Cu at (229.4, 79.0)
- added D56: , ComboDiode, F.Cu at (219.9, 60.0)
- added D57: , ComboDiode, F.Cu at (238.9, 155.0)
- added D58: , ComboDiode, F.Cu at (248.4, 136.0)
- added D59: , ComboDiode, F.Cu at (248.4, 117.0)
- added D6: , ComboDiode, F.Cu at (25.0, 60.0)
- added D60: , ComboDiode, F.Cu at (248.4, 98.0)
- added D61: , ComboDiode, F.Cu at (248.4, 79.0)
- added D62: , ComboDiode, F.Cu at (257.9, 155.0)
- added D63: , ComboDiode, F.Cu at (276.9, 136.0)
- added D64: , ComboDiode, F.Cu at (267.4, 117.0)
- added D65: , ComboDiode, F.Cu at (267.4, 98.0)
- added D66: , ComboDiode, F.Cu at (267.4, 79.0)
- added D67: , ComboDiode, F.Cu at (257.9, 60.0)
- added D68: , ComboDiode, F.Cu at (276.9, 155.0)
- added D69: , ComboDiode, F.Cu at (295.9, 117.0)
- added D7: , ComboDiode, F.Cu at (44.0, 155.0)
- added D70: , ComboDiode, F.Cu at (286.4, 98.0)
- added D71: , ComboDiode, F.Cu at (286.4, 79.0)
- added D72: , ComboDiode, F.Cu at (276.9, 60.0)
- added D73: , ComboDiode, F.Cu at (305.4, 98.0)
- added D74: , ComboDiode, F.Cu at (314.9, 79.0)
- added D75: , ComboDiode, F.Cu at (295.9, 60.0)
- added D76: , ComboDiode, F.Cu at (314.9, 60.0)
- added D77: , ComboDiode, F.Cu at (334.0, 151.6)
- added D78: , ComboDiode, F.Cu at (320.6, 138.2)
- added D79: , ComboDiode, F.Cu at (347.5, 138.2)
- added D8: , ComboDiode, F.Cu at (53.5, 136.0)
- added D80: , ComboDiode, F.Cu at (334.0, 124.8)
- added D81: , ComboDiode, F.Cu at (375.1, 129.4)
- added D82: , ComboDiode, F.Cu at (361.7, 116.0)
- added D83: , ComboDiode, F.Cu at (388.5, 116.0)
- added D84: , ComboDiode, F.Cu at (375.1, 102.6)
- added D85: , ComboDiode, F.Cu at (353.0, 79.0)
- added D86: , ComboDiode, F.Cu at (353.0, 60.0)
- added D87: , ComboDiode, F.Cu at (372.0, 79.0)
- added D88: , ComboDiode, F.Cu at (372.0, 60.0)
- added D89: , ComboDiode, F.Cu at (391.0, 79.0)
- added D9: , ComboDiode, F.Cu at (53.5, 117.0)
- added D90: , ComboDiode, F.Cu at (391.0, 60.0)
- added MCU1: , ProMicro, F.Cu at (141.4, 59.0)
- added S1: , MX, F.Cu at (25.0, 150.0)
- added S10: , MX, F.Cu at (53.5, 93.0)
- added S11: , MX, F.Cu at (44.0, 74.0)
- added S12: , MX, F.Cu at (63.0, 150.0)
- added S13: , MX, F.Cu at (72.5, 131.0)
- added S14: , MX, F.Cu at (72.5, 112.0)
- added S15: , MX, F.Cu at (72.5, 93.0)
- added S16: , MX, F.Cu at (63.0, 74.0)
- added S17: , MX, F.Cu at (63.0, 55.0)
- added S18: , MX, F.Cu at (82.0, 150.0)
- added S19: , MX, F.Cu at (91.5, 131.0)
- added S2: , MX, F.Cu at (25.0, 131.0)
- added S20: , MX, F.Cu at (91.5, 112.0)
- added S21: , MX, F.Cu at (91.5, 93.0)
- added S22: , MX, F.Cu at (82.0, 74.0)
- added S23: , MX, F.Cu at (82.0, 55.0)
- added S24: , MX, F.Cu at (120.0, 150.0)
- added S25: , MX, F.Cu at (110.5, 131.0)
- added S26: , MX, F.Cu at (110.5, 112.0)
- added S27: , MX, F.Cu at (110.5, 93.0)
- added S28: , MX, F.Cu at (101.0, 74.0)
- added S29: , MX, F.Cu at (101.0, 55.0)
- added S3: , MX, F.Cu at (25.0, 112.0)
- added S30: , MX, F.Cu at (129.5, 131.0)
- added S31: , MX, F.Cu at (129.5, 112.0)
- added S32: , MX, F.Cu at (129.5, 93.0)
- added S33: , MX, F.Cu at (120.0, 74.0)
- added S34: , MX, F.Cu at (120.0, 55.0)
- added S35: , MX, F.Cu at (181.9, 150.0)
- added S36: , MX, F.Cu at (172.4, 131.0)
- added S37: , MX, F.Cu at (172.4, 112.0)
- added S38: , MX, F.Cu at (172.4, 93.0)
- added S39: , MX, F.Cu at (172.4, 74.0)
- added S4: , MX, F.Cu at (25.0, 93.0)
- added S40: , MX, F.Cu at (162.9, 55.0)
- added S41: , MX, F.Cu at (191.4, 131.0)
- added S42: , MX, F.Cu at (191.4, 112.0)
- added S43: , MX, F.Cu at (191.4, 93.0)
- added S44: , MX, F.Cu at (191.4, 74.0)
- added S45: , MX, F.Cu at (181.9, 55.0)
- added S46: , MX, F.Cu at (210.4, 131.0)
- added S47: , MX, F.Cu at (210.4, 112.0)
- added S48: , MX, F.Cu at (210.4, 93.0)
- added S49: , MX, F.Cu at (210.4, 74.0)
- added S5: , MX, F.Cu at (25.0, 74.0)
- added S50: , MX, F.Cu at (200.9, 55.0)
- added S51: , MX, F.Cu at (219.9, 150.0)
- added S52: , MX, F.Cu at (229.4, 131.0)
- added S53: , MX, F.Cu at (229.4, 112.0)
- added S54: , MX, F.Cu at (229.4, 93.0)
- added S55: , MX, F.Cu at (229.4, 74.0)
- added S56: , MX, F.Cu at (219.9, 55.0)
- added S57: , MX, F.Cu at (238.9, 150.0)
- added S58: , MX, F.Cu at (248.4, 131.0)
- added S59: , MX, F.Cu at (248.4, 112.0)
- added S6: , MX, F.Cu at (25.0, 55.0)
- added S60: , MX, F.Cu at (248.4, 93.0)
- added S61: , MX, F.Cu at (248.4, 74.0)
- added S62: , MX, F.Cu at (257.9, 150.0)
- added S63: , MX, F.Cu at (276.9, 131.0)
- added S64: , MX, F.Cu at (267.4, 112.0)
- added S65: , MX, F.Cu at (267.4, 93.0)
- added S66: , MX, F.Cu at (267.4, 74.0)
- added S67: , MX, F.Cu at (257.9, 55.0)
- added S68: , MX, F.Cu at (276.9, 150.0)
- added S69: , MX, F.Cu at (295.9, 112.0)
- added S7: , MX, F.Cu at (44.0, 150.0)
- added S70: , MX, F.Cu at (286.4, 93.0)
- added S71: , MX, F.Cu at (286.4, 74.0)
- added S72: , MX, F.Cu at (276.9, 55.0)
- added S73: , MX, F.Cu at (305.4, 93.0)
- added S74: , MX, F.Cu at (314.9, 74.0)
- added S75: , MX, F.Cu at (295.9, 55.0)
- added S76: , MX, F.Cu at (314.9, 55.0)
- added S77: , MX, F.Cu at (330.5, 148.1)
- added S78: , MX, F.Cu at (317.1, 134.7)
- added S79: , MX, F.Cu at (343.9, 134.7)
- added S8: , MX, F.Cu at (53.5, 131.0)
- added S80: , MX, F.Cu at (330.5, 121.2)
- added S81: , MX, F.Cu at (371.6, 125.9)
- added S82: , MX, F.Cu at (358.1, 112.5)
- added S83: , MX, F.Cu at (385.0, 112.5)
- added S84: , MX, F.Cu at (371.6, 99.0)
- added S85: , MX, F.Cu at (353.0, 74.0)
- added S86: , MX, F.Cu at (353.0, 55.0)
- added S87: , MX, F.Cu at (372.0, 74.0)
- added S88: , MX, F.Cu at (372.0, 55.0)
- added S89: , MX, F.Cu at (391.0, 74.0)
- added S9: , MX, F.Cu at (53.5, 112.0)
- added S90: , MX, F.Cu at (391.0, 55.0)
Other:
- board size 384.2 x 120.8 mm -> 388.9 x 120.8 mm

Commit message: reset button
Parts:
- added B1: , E73:SW_TACT_ALPS_SKQGABE010, F.Cu at (336.9, 80.0)
- moved D1 25.2 mm to (28.0, 180.0)
- moved D10 25.2 mm to (56.5, 123.0)
- moved D11 25.2 mm to (47.0, 104.0)
- moved D12 25.2 mm to (66.0, 180.0)
- moved D13 25.2 mm to (75.5, 161.0)
- moved D14 25.2 mm to (75.5, 142.0)
- moved D15 25.2 mm to (75.5, 123.0)
- moved D16 25.2 mm to (66.0, 104.0)
- moved D17 25.2 mm to (66.0, 85.0)
- moved D18 25.2 mm to (85.0, 180.0)
- moved D19 25.2 mm to (94.5, 161.0)
- moved D2 25.2 mm to (28.0, 161.0)
- moved D20 25.2 mm to (94.5, 142.0)
- moved D21 25.2 mm to (94.5, 123.0)
- moved D22 25.2 mm to (85.0, 104.0)
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
Commit message: added case holes
Parts:
- added REF**: RollerEncoder_Panasonic_EVQWGD001, RollerEncoder_Panasonic_EVQWGD001, F.Cu at (153.0, 118.0)
- added ROT1: , rotary_encoder, F.Cu at (153.0, 156.0)
- added _1: , MountingHole_2.2mm_M2_Pad_Via, F.Cu at (46.0, 74.3)
- added _2: , MountingHole_2.2mm_M2_Pad_Via, F.Cu at (383.5, 85.7)
- added _3: , MountingHole_2.2mm_M2_Pad_Via, F.Cu at (307.9, 179.3)
- added _4: , MountingHole_2.2mm_M2_Pad_Via, F.Cu at (41.3, 161.7)
- moved B1 1.00 mm to (335.9, 80.0), turned to -45 degrees
- moved D1 1.00 mm to (27.0, 180.0)
- moved D10 1.00 mm to (55.5, 123.0)
- moved D11 1.00 mm to (46.0, 104.0)
- moved D12 1.00 mm to (65.0, 180.0)
- moved D13 1.00 mm to (74.5, 161.0)
- moved D14 1.00 mm to (74.5, 142.0)
- moved D15 1.00 mm to (74.5, 123.0)
- moved D16 1.00 mm to (65.0, 104.0)
- moved D17 1.00 mm to (65.0, 85.0)
- moved D18 1.00 mm to (84.0, 180.0)
- moved D19 1.00 mm to (93.5, 161.0)
- moved D2 1.00 mm to (27.0, 161.0)
- moved D20 1.00 mm to (93.5, 142.0)
- moved D21 1.00 mm to (93.5, 123.0)
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Connections:
- D77 pad 2: one_a -> left_bottom
- D78 pad 2: one_b -> left_top
- D79 pad 2: two_a -> right_bottom
- D80 pad 2: two_b -> right_top
- D81 pad 2: one_a -> left_bottom
- D82 pad 2: one_b -> left_top
- D83 pad 2: two_a -> right_bottom
- D84 pad 2: two_b -> right_top
- S77 pad 2: one_a -> left_bottom
- S78 pad 2: one_b -> left_top
- S79 pad 2: two_a -> right_bottom
- S80 pad 2: two_b -> right_top
- S81 pad 2: one_a -> left_bottom
- S82 pad 2: one_b -> left_top
- S83 pad 2: two_a -> right_bottom
- S84 pad 2: two_b -> right_top
Other:
- board size 388.9 x 120.8 mm -> 390.9 x 123.2 mm

Commit message: moved case holes
Parts:
- moved _2 3.80 mm to (383.5, 89.5)
- moved MCU1 3.25 mm to (143.4, 87.2)
- turned ROT1 to -90 degrees
Changed lines of the file:
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@@
     )
       (module ProMicro (layer F.Cu)
-      (at 143.43124999999998 84 -90)
+      (at 143.43124999999998 87.25 -90)
       (fp_text reference "MCU1" (at 0 0) (layer F.SilkS) hide (effects (font (size 1.27 1.27) (thickness 0.15))))
       (fp_text value "" (at 0 0) (layer F.SilkS) hide (effects (font (size 1.27 1.27) (thickness 0.15))))
@@
         )
         (module rotary_encoder (layer F.Cu)
-            (at 152.95625 156 -45)
+            (at 152.95625 156 -90)
             (fp_text reference "ROT1" (at 0 0.5) (layer F.SilkS)
                 hide (effects (font (size 1 1) (thickness 0.15))))
@@
             (fp_circle (center -0.12 -0.04) (end 2.88 -0.04) (layer F.SilkS) (width 0.12))
             (fp_circle (center -0.12 -0.04) (end 2.88 -0.04) (layer F.Fab) (width 0.12))
-            (pad A thru_hole rect (at -7.62 -2.54 -45) (size 2 2) (drill 1) (layers *.Cu *.Mask) (net 52 "GND"))
+            (pad A thru_hole rect (at -7.62 -2.54 -90) (size 2 2) (drill 1) (layers *.Cu *.Mask) (net 52 "GND"))
             (pad C thru_hole circle (at -7.62 -0.04) (size 2 2) (drill 1) (layers *.Cu *.Mask) (net 52 "GND"))
             (pad B thru_hole circle (at -7.62 2.46) (size 2 2) (drill 1) (layers *.Cu *.Mask) (net 52 "GND"))
             (pad 1 thru_hole circle (at 6.88 -2.54) (size 1.5 1.5) (drill 1) (layers *.Cu *.Mask) (net 52 "GND"))
             (pad 2 thru_hole circle (at 6.88 2.46) (size 1.5 1.5) (drill 1) (layers *.Cu *.Mask) (net 52 "GND"))
-            (pad "" thru_hole rect (at -0.12 -5.64 -45) (size 3.2 2) (drill oval 2.8 1.5) (layers *.Cu *.Mask))
-            (pad "" thru_hole rect (at -0.12 5.56 -45)  (size 3.2 2) (drill oval 2.8 1.5) (layers *.Cu *.Mask))
+            (pad "" thru_hole rect (at -0.12 -5.64 -90) (size 3.2 2) (drill oval 2.8 1.5) (layers *.Cu *.Mask))
+            (pad "" thru_hole rect (at -0.12 5.56 -90)  (size 3.2 2) (drill oval 2.8 1.5) (layers *.Cu *.Mask))
         )
     (module "MountingHole_2.2mm_M2_Pad_Via" (version 20210722) (generator pcbnew) (layer "F.Cu")
@@
     )
     (module "MountingHole_2.2mm_M2_Pad_Via" (version 20210722) (generator pcbnew) (layer "F.Cu")
-      (at 383.46250000000003 85.7 0)
+      (at 383.46250000000003 89.5 0)
       (fp_text reference "_2" (at 0 -3.2) (layer "F.SilkS") hide
         (effects (font (size 1 1) (thickness 0.15)))

Commit message: added todos
Connections:
- REF** pad D: GND -> (no net)
Changed lines of the file:
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@@
           (pad B thru_hole circle (at -5.625 -1.27 0) (size 1.6 1.6) (drill 0.9) (layers *.Cu *.Mask) (net 52 "GND"))
           (pad C thru_hole circle (at -5.625 1.27 0) (size 1.6 1.6) (drill 0.9) (layers *.Cu *.Mask) (net 52 "GND"))
-          (pad D thru_hole circle (at -5.625 3.81 0) (size 1.6 1.6) (drill 0.9) (layers *.Cu *.Mask) (net 52 "GND"))
+          (pad D thru_hole circle (at -5.625 3.81 0) (size 1.6 1.6) (drill 0.9) (layers *.Cu *.Mask) (net 0 ""))
           (pad "" np_thru_hole circle (at -5.625 6.3 0) (size 1.5 1.5) (drill 1.5) (layers *.Cu *.Mask))
         )

Commit message: init node
Parts:
- removed _1, _2, _3, _4: , MountingHole_2.2mm_M2_Pad_Via
- moved D85 14.3 mm to (340.7, 104.0)
- moved D86 14.3 mm to (340.7, 85.0)
- moved D87 14.3 mm to (359.7, 104.0)
- moved D88 14.3 mm to (359.7, 85.0)
- moved D89 14.3 mm to (378.7, 104.0)
- moved D90 14.3 mm to (378.7, 85.0)
- moved S85 14.3 mm to (340.7, 99.0)
- moved S86 14.3 mm to (340.7, 80.0)
- moved S87 14.3 mm to (359.7, 99.0)
- moved S88 14.3 mm to (359.7, 80.0)
- moved S89 14.3 mm to (378.7, 99.0)
- moved S90 14.3 mm to (378.7, 80.0)
- moved D77 10.5 mm to (325.6, 176.6)
- moved D78 10.5 mm to (312.1, 163.2)
- moved D79 10.5 mm to (339.0, 163.2)
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Other:
- board size 390.9 x 123.2 mm -> 379.6 x 123.2 mm
