File: output/pcbs/tutorial.kicad_pcb (KiCad board)
At the start: 2 copper layers, 379.6 x 123.2 mm, 185 parts

Commit message: updated keys to ortho
Parts:
- added DIP2: DIP-16_W7.62mm_Socket, DIP-16_W7.62mm_Socket, F.Cu at (254.0, 69.1)
- moved D68 95.3 mm to (276.9, 84.7)
- moved S68 95.3 mm to (276.9, 79.7)
- moved D57 95.3 mm to (238.8, 84.7)
- moved S57 95.3 mm to (238.8, 79.7)
- moved D51 95.3 mm to (219.7, 84.7)
- moved S51 95.3 mm to (219.7, 79.7)
- moved D62 76.2 mm to (257.8, 103.8)
- moved S62 76.2 mm to (257.8, 98.8)
- moved D67 28.7 mm to (276.9, 103.8)
- moved S67 28.7 mm to (276.9, 98.8)
- moved D56 28.7 mm to (238.8, 103.8)
- moved S56 28.7 mm to (238.8, 98.8)
- moved D50 28.6 mm to (219.7, 103.8)
- moved S50 28.6 mm to (219.7, 98.8)
- moved D64 25.9 mm to (282.2, 160.9)
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Connections:
- D46 pad 2: middle_bottom -> middle_mod
- D47 pad 2: middle_home -> middle_bottom
- D48 pad 2: middle_top -> middle_home
- D49 pad 2: middle_num -> middle_top
- D50 pad 2: middle_func -> middle_num
- D51 pad 2: ring_mod -> middle_func
- D52 pad 2: ring_bottom -> ring_mod
- D53 pad 2: ring_home -> ring_bottom
- D54 pad 2: ring_top -> ring_home
- D55 pad 2: ring_num -> ring_top
- D56 pad 2: ring_func -> ring_num
- D57 pad 2: pinky_mod -> ring_func
- D58 pad 2: pinky_bottom -> pinky_mod
- D59 pad 2: pinky_home -> pinky_bottom
- D60 pad 2: pinky_top -> pinky_home
- D61 pad 2: pinky_num -> pinky_top
- D62 pad 2: outer_mod -> pinky_num
- D63 pad 2: outer_bottom -> outer_mod
- D64 pad 2: outer_home -> outer_bottom
- D65 pad 2: outer_top -> outer_home
- D66 pad 2: outer_num -> outer_top
- D67 pad 2: outer_func -> outer_num
- D68 pad 2: outer2_mod -> outer_func
- S46 pad 2: middle_bottom -> middle_mod
- S47 pad 2: middle_home -> middle_bottom
- S48 pad 2: middle_top -> middle_home
- S49 pad 2: middle_num -> middle_top
- S50 pad 2: middle_func -> middle_num
- S51 pad 2: ring_mod -> middle_func
- S52 pad 2: ring_bottom -> ring_mod
- S53 pad 2: ring_home -> ring_bottom
- S54 pad 2: ring_top -> ring_home
- S55 pad 2: ring_num -> ring_top
- S56 pad 2: ring_func -> ring_num
- S57 pad 2: pinky_mod -> ring_func
- S58 pad 2: pinky_bottom -> pinky_mod
- S59 pad 2: pinky_home -> pinky_bottom
- S60 pad 2: pinky_top -> pinky_home
- S61 pad 2: pinky_num -> pinky_top
- S62 pad 2: outer_mod -> pinky_num
- S63 pad 2: outer_bottom -> outer_mod
- S64 pad 2: outer_home -> outer_bottom
- S65 pad 2: outer_top -> outer_home
- S66 pad 2: outer_num -> outer_top
- S67 pad 2: outer_func -> outer_num
- S68 pad 2: outer2_mod -> outer_func
Other:
- board size 379.6 x 123.2 mm -> 410.2 x 131 mm
