File: output/pcbs/travis_erg2024.kicad_pcb-wired.kicad_pcb (KiCad board)
At the start: 2 copper layers, 393.3 x 146.1 mm, 380 parts, among them SW1 SW_PUSH_6mm_H4.3mm

Commit message: wiring
Parts:
- moved C90 0.33 mm to (57.9, 64.5)
- moved C91 0.17 mm to (270.2, 64.8)
Connections:
- MCU1 pad 21: scrA -> scrC
- MCU1 pad 22: scrB -> scrA
Routing:
- net row3: track 0.00 -> 534.3 mm
- net row4: track 0.00 -> 497.6 mm, vias 0 -> 1
- net row1: track 0.00 -> 490.4 mm, vias 0 -> 2
- net row2: track 0.00 -> 485.1 mm, vias 0 -> 3
- net row5: track 0.00 -> 484.7 mm
- net row0: track 0.00 -> 465.1 mm, vias 0 -> 1
- net col15: track 0.00 -> 284.5 mm, vias 0 -> 7
- net mux3: track 0.00 -> 278.2 mm, vias 0 -> 1
- net col4: track 0.00 -> 268.8 mm, vias 0 -> 10
- net col14: track 0.00 -> 268.5 mm, vias 0 -> 7
- net mux2: track 0.00 -> 259.7 mm, vias 0 -> 2
- net mux1: track 0.00 -> 253.8 mm, vias 0 -> 2
- net mux0: track 0.00 -> 240.8 mm, vias 0 -> 2
- net col2: track 0.00 -> 240.4 mm, vias 0 -> 10
- net col1: track 0.00 -> 237.9 mm, vias 0 -> 9
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