File: output/pcbs/travis_erg2024-new3.kicad_pcb (KiCad board)
At the start: 2 copper layers, 385.3 x 144.8 mm, 378 parts, among them SW1 SW_PUSH_6mm_H4.3mm

Commit message: updating routes
Parts:
- removed the C1 at (44.3, 207.9)
- removed C10, C11, C12, C13, C14, C15, C16, C17, C18, C19, C20, C21, C22, C23, C24, C25, C26, C27, C28, C29, C30, C31, C32, C33, C34, C35, C36, C37, C38, C39, C4, C40, C41, C42, C43, C44, C45, C46, C47, C48, C49, C5, C50, C51, C52, C53, C54, C55, C56, C57, C58, C59, C6, C60, C61, C62, C63, C64, C65, C66, C67, C68, C69, C7, C70, C71, C72, C73, C74, C75, C76, C77, C78, C79, C8, C80, C81, C82, C83, C84, C85, C86, C87, C88, C9: 104, travis:C_Disc_D4.7mm_W2.5mm_P5.00mm
- removed the C2 at (38.7, 169.9)
- removed the C3 at (43.7, 131.7)
- removed the D1 at (50.2, 191.5)
- removed D10, D11, D12, D13, D14, D15, D16, D17, D18, D19, D20, D21, D22, D23, D24, D25, D26, D27, D28, D29, D3, D30, D31, D32, D33, D34, D35, D36, D37, D38, D39, D4, D40, D41, D42, D43, D44, D45, D46, D47, D48, D49, D5, D50, D51, D52, D53, D54, D55, D56, D57, D58, D59, D6, D60, D61, D62, D63, D64, D65, D66, D67, D68, D69, D7, D70, D71, D72, D73, D74, D75, D76, D77, D78, D79, D8, D80, D81, D82, D83, D84, D85, D86, D87, D88, D9: 1N4148, travis:Diode_DO-35
- removed the D2 at (44.6, 153.5)
- removed LED1, LED10, LED11, LED12, LED13, LED14, LED15, LED16, LED17, LED18, LED19, LED2, LED20, LED21, LED22, LED23, LED24, LED25, LED26, LED27, LED28, LED29, LED3, LED30, LED31, LED32, LED33, LED34, LED35, LED36, LED37, LED38, LED39, LED4, LED40, LED41, LED42, LED43, LED44, LED45, LED46, LED47, LED48, LED49, LED5, LED50, LED51, LED52, LED53, LED54, LED55, LED56, LED57, LED58, LED59, LED6, LED60, LED61, LED62, LED63, LED64, LED65, LED66, LED67, LED68, LED69, LED7, LED70, LED71, LED72, LED73, LED74, LED75, LED76, LED77, LED78, LED79, LED8, LED80, LED81, LED82, LED83, LED84, LED85, LED86, LED87, LED88, LED9: SK6812mini-e, travis:led_SK6812mini-e (per-key single-side)
- removed S1, S10, S11, S12, S13, S14, S15, S16, S17, S18, S19, S2, S20, S21, S22, S23, S24, S25, S26, S27, S28, S29, S3, S30, S31, S32, S33, S34, S35, S36, S37, S38, S39, S4, S40, S41, S42, S43, S44, S45, S46, S47, S48, S49, S5, S50, S51, S52, S53, S54, S55, S56, S57, S58, S59, S6, S60, S61, S62, S63, S64, S65, S66, S67, S68, S69, S7, S70, S71, S72, S73, S74, S75, S76, S77, S78, S79, S8, S80, S81, S82, S83, S84, S85, S86, S87, S88, S9: Kailh MX Switch Sockets, travis:MX
- added KC1: 104, travis:C_Disc_D4.7mm_W2.5mm_P5.00mm, B.Cu at (44.3, 207.9)
- added KC10: 104, travis:C_Disc_D4.7mm_W2.5mm_P5.00mm, B.Cu at (101.2, 204.8)
- added KC11: 104, travis:C_Disc_D4.7mm_W2.5mm_P5.00mm, B.Cu at (102.2, 166.8)
- added KC12: 104, travis:C_Disc_D4.7mm_W2.5mm_P5.00mm, B.Cu at (103.2, 128.7)
- added KC13: 104, travis:C_Disc_D4.7mm_W2.5mm_P5.00mm, B.Cu at (121.7, 168.3)
- added KC14: 104, travis:C_Disc_D4.7mm_W2.5mm_P5.00mm, B.Cu at (123.4, 130.2)
- added KC15: 104, travis:C_Disc_D4.7mm_W2.5mm_P5.00mm, B.Cu at (137.5, 207.4)
- added KC16: 104, travis:C_Disc_D4.7mm_W2.5mm_P5.00mm, B.Cu at (140.8, 169.4)
- added KC17: 104, travis:C_Disc_D4.7mm_W2.5mm_P5.00mm, B.Cu at (142.7, 131.4)
- added KC18: 104, travis:C_Disc_D4.7mm_W2.5mm_P5.00mm, B.Cu at (193.8, 207.1)
- added KC19: 104, travis:C_Disc_D4.7mm_W2.5mm_P5.00mm, B.Cu at (190.4, 169.2)
- added KC2: 104, travis:C_Disc_D4.7mm_W2.5mm_P5.00mm, B.Cu at (38.7, 169.9)
- added KC20: 104, travis:C_Disc_D4.7mm_W2.5mm_P5.00mm, B.Cu at (188.6, 131.1)
- added KC21: 104, travis:C_Disc_D4.7mm_W2.5mm_P5.00mm, B.Cu at (209.5, 168.0)
- added KC22: 104, travis:C_Disc_D4.7mm_W2.5mm_P5.00mm, B.Cu at (207.6, 129.9)
- added KC23: 104, travis:C_Disc_D4.7mm_W2.5mm_P5.00mm, B.Cu at (230.1, 204.2)
- added KC24: 104, travis:C_Disc_D4.7mm_W2.5mm_P5.00mm, B.Cu at (229.0, 166.1)
- added KC25: 104, travis:C_Disc_D4.7mm_W2.5mm_P5.00mm, B.Cu at (227.8, 128.0)
- added KC26: 104, travis:C_Disc_D4.7mm_W2.5mm_P5.00mm, B.Cu at (249.0, 204.7)
- added KC27: 104, travis:C_Disc_D4.7mm_W2.5mm_P5.00mm, B.Cu at (248.5, 166.6)
- added KC28: 104, travis:C_Disc_D4.7mm_W2.5mm_P5.00mm, B.Cu at (248.0, 128.5)
- added KC29: 104, travis:C_Disc_D4.7mm_W2.5mm_P5.00mm, B.Cu at (268.0, 206.5)
- added KC3: 104, travis:C_Disc_D4.7mm_W2.5mm_P5.00mm, B.Cu at (43.7, 131.7)
- added KC30: 104, travis:C_Disc_D4.7mm_W2.5mm_P5.00mm, B.Cu at (268.1, 168.4)
- added KC31: 104, travis:C_Disc_D4.7mm_W2.5mm_P5.00mm, B.Cu at (268.3, 130.3)
- added KC32: 104, travis:C_Disc_D4.7mm_W2.5mm_P5.00mm, B.Cu at (287.0, 206.5)
- added KC33: 104, travis:C_Disc_D4.7mm_W2.5mm_P5.00mm, B.Cu at (287.2, 168.4)
- added KC34: 104, travis:C_Disc_D4.7mm_W2.5mm_P5.00mm, B.Cu at (287.4, 130.3)
- added KC35: 104, travis:C_Disc_D4.7mm_W2.5mm_P5.00mm, B.Cu at (311.6, 168.5)
- added KC36: 104, travis:C_Disc_D4.7mm_W2.5mm_P5.00mm, B.Cu at (306.4, 130.4)
- added KC37: 104, travis:C_Disc_D4.7mm_W2.5mm_P5.00mm, B.Cu at (330.8, 130.5)
- added KC38: 104, travis:C_Disc_D4.7mm_W2.5mm_P5.00mm, B.Cu at (344.9, 212.0)
- added KC39: 104, travis:C_Disc_D4.7mm_W2.5mm_P5.00mm, B.Cu at (357.8, 197.9)
- added KC4: 104, travis:C_Disc_D4.7mm_W2.5mm_P5.00mm, B.Cu at (63.4, 207.8)
- added KC40: 104, travis:C_Disc_D4.7mm_W2.5mm_P5.00mm, B.Cu at (373.8, 180.3)
- added KC41: 104, travis:C_Disc_D4.7mm_W2.5mm_P5.00mm, B.Cu at (386.6, 166.2)
- added KC42: 104, travis:C_Disc_D4.7mm_W2.5mm_P5.00mm, B.Cu at (373.1, 130.7)
- added KC43: 104, travis:C_Disc_D4.7mm_W2.5mm_P5.00mm, B.Cu at (392.1, 130.8)
- added KC44: 104, travis:C_Disc_D4.7mm_W2.5mm_P5.00mm, B.Cu at (33.9, 189.0)
- added KC45: 104, travis:C_Disc_D4.7mm_W2.5mm_P5.00mm, B.Cu at (33.6, 150.9)
- added KC46: 104, travis:C_Disc_D4.7mm_W2.5mm_P5.00mm, B.Cu at (38.5, 112.7)
- added KC47: 104, travis:C_Disc_D4.7mm_W2.5mm_P5.00mm, B.Cu at (58.2, 188.7)
- added KC48: 104, travis:C_Disc_D4.7mm_W2.5mm_P5.00mm, B.Cu at (57.9, 150.7)
- added KC49: 104, travis:C_Disc_D4.7mm_W2.5mm_P5.00mm, B.Cu at (77.4, 186.5)
- added KC5: 104, travis:C_Disc_D4.7mm_W2.5mm_P5.00mm, B.Cu at (63.0, 169.7)
- added KC50: 104, travis:C_Disc_D4.7mm_W2.5mm_P5.00mm, B.Cu at (77.8, 148.4)
- added KC51: 104, travis:C_Disc_D4.7mm_W2.5mm_P5.00mm, B.Cu at (78.1, 110.3)
- added KC52: 104, travis:C_Disc_D4.7mm_W2.5mm_P5.00mm, B.Cu at (96.7, 185.7)
- added KC53: 104, travis:C_Disc_D4.7mm_W2.5mm_P5.00mm, B.Cu at (97.7, 147.6)
- added KC54: 104, travis:C_Disc_D4.7mm_W2.5mm_P5.00mm, B.Cu at (98.7, 109.5)
- added KC55: 104, travis:C_Disc_D4.7mm_W2.5mm_P5.00mm, B.Cu at (115.9, 187.1)
- added KC56: 104, travis:C_Disc_D4.7mm_W2.5mm_P5.00mm, B.Cu at (117.5, 149.1)
- added KC57: 104, travis:C_Disc_D4.7mm_W2.5mm_P5.00mm, B.Cu at (119.2, 111.0)
- added KC58: 104, travis:C_Disc_D4.7mm_W2.5mm_P5.00mm, B.Cu at (134.9, 188.2)
- added KC59: 104, travis:C_Disc_D4.7mm_W2.5mm_P5.00mm, B.Cu at (136.8, 150.1)
- added KC6: 104, travis:C_Disc_D4.7mm_W2.5mm_P5.00mm, B.Cu at (62.7, 131.6)
- added KC60: 104, travis:C_Disc_D4.7mm_W2.5mm_P5.00mm, B.Cu at (138.6, 112.1)
- added KC61: 104, travis:C_Disc_D4.7mm_W2.5mm_P5.00mm, B.Cu at (186.4, 188.4)
- added KC62: 104, travis:C_Disc_D4.7mm_W2.5mm_P5.00mm, B.Cu at (184.5, 150.4)
- added KC63: 104, travis:C_Disc_D4.7mm_W2.5mm_P5.00mm, B.Cu at (182.7, 112.3)
- added KC64: 104, travis:C_Disc_D4.7mm_W2.5mm_P5.00mm, B.Cu at (205.4, 187.3)
- added KC65: 104, travis:C_Disc_D4.7mm_W2.5mm_P5.00mm, B.Cu at (203.5, 149.2)
- added KC66: 104, travis:C_Disc_D4.7mm_W2.5mm_P5.00mm, B.Cu at (201.7, 111.2)
- added KC67: 104, travis:C_Disc_D4.7mm_W2.5mm_P5.00mm, B.Cu at (224.5, 185.3)
- added KC68: 104, travis:C_Disc_D4.7mm_W2.5mm_P5.00mm, B.Cu at (223.4, 147.2)
- added KC69: 104, travis:C_Disc_D4.7mm_W2.5mm_P5.00mm, B.Cu at (222.2, 109.1)
- added KC7: 104, travis:C_Disc_D4.7mm_W2.5mm_P5.00mm, B.Cu at (82.3, 205.6)
- added KC70: 104, travis:C_Disc_D4.7mm_W2.5mm_P5.00mm, B.Cu at (243.8, 185.7)
- added KC71: 104, travis:C_Disc_D4.7mm_W2.5mm_P5.00mm, B.Cu at (243.3, 147.6)
- added KC72: 104, travis:C_Disc_D4.7mm_W2.5mm_P5.00mm, B.Cu at (242.8, 109.5)
- added KC73: 104, travis:C_Disc_D4.7mm_W2.5mm_P5.00mm, B.Cu at (263.1, 187.4)
- added KC74: 104, travis:C_Disc_D4.7mm_W2.5mm_P5.00mm, B.Cu at (263.2, 149.3)
- added KC75: 104, travis:C_Disc_D4.7mm_W2.5mm_P5.00mm, B.Cu at (287.5, 187.5)
- added KC76: 104, travis:C_Disc_D4.7mm_W2.5mm_P5.00mm, B.Cu at (282.3, 149.4)
- added KC77: 104, travis:C_Disc_D4.7mm_W2.5mm_P5.00mm, B.Cu at (282.4, 111.3)
- added KC78: 104, travis:C_Disc_D4.7mm_W2.5mm_P5.00mm, B.Cu at (301.3, 149.4)
- added KC79: 104, travis:C_Disc_D4.7mm_W2.5mm_P5.00mm, B.Cu at (301.5, 111.3)
- added KC8: 104, travis:C_Disc_D4.7mm_W2.5mm_P5.00mm, B.Cu at (82.6, 167.5)
- added KC80: 104, travis:C_Disc_D4.7mm_W2.5mm_P5.00mm, B.Cu at (320.4, 149.5)
- added KC81: 104, travis:C_Disc_D4.7mm_W2.5mm_P5.00mm, B.Cu at (320.5, 111.4)
- added KC82: 104, travis:C_Disc_D4.7mm_W2.5mm_P5.00mm, B.Cu at (339.6, 111.5)
- added KC83: 104, travis:C_Disc_D4.7mm_W2.5mm_P5.00mm, B.Cu at (327.5, 202.9)
- added KC84: 104, travis:C_Disc_D4.7mm_W2.5mm_P5.00mm, B.Cu at (340.3, 188.8)
- added KC85: 104, travis:C_Disc_D4.7mm_W2.5mm_P5.00mm, B.Cu at (356.3, 171.2)
- added KC86: 104, travis:C_Disc_D4.7mm_W2.5mm_P5.00mm, B.Cu at (369.1, 157.1)
- added KC87: 104, travis:C_Disc_D4.7mm_W2.5mm_P5.00mm, B.Cu at (368.2, 111.6)
- added KC88: 104, travis:C_Disc_D4.7mm_W2.5mm_P5.00mm, B.Cu at (387.2, 111.7)
- added KC9: 104, travis:C_Disc_D4.7mm_W2.5mm_P5.00mm, B.Cu at (82.9, 129.4)
- added KD1: 1N4148, travis:Diode_DO-35, B.Cu at (50.2, 191.5)
- added KD10: 1N4148, travis:Diode_DO-35, B.Cu at (107.6, 188.7)
- added KD11: 1N4148, travis:Diode_DO-35, B.Cu at (108.6, 150.6)
- added KD12: 1N4148, travis:Diode_DO-35, B.Cu at (109.6, 112.5)
- added KD13: 1N4148, travis:Diode_DO-35, B.Cu at (128.4, 152.3)
- added KD14: 1N4148, travis:Diode_DO-35, B.Cu at (130.1, 114.2)
- added KD15: 1N4148, travis:Diode_DO-35, B.Cu at (144.3, 191.4)
- added KD16: 1N4148, travis:Diode_DO-35, B.Cu at (147.6, 153.4)
- added KD17: 1N4148, travis:Diode_DO-35, B.Cu at (149.5, 115.3)
- added KD18: 1N4148, travis:Diode_DO-35, B.Cu at (199.0, 190.6)
- added KD19: 1N4148, travis:Diode_DO-35, B.Cu at (195.7, 152.6)
- added KD2: 1N4148, travis:Diode_DO-35, B.Cu at (44.6, 153.5)
- added KD20: 1N4148, travis:Diode_DO-35, B.Cu at (193.8, 114.5)
- added KD21: 1N4148, travis:Diode_DO-35, B.Cu at (214.7, 151.4)
- added KD22: 1N4148, travis:Diode_DO-35, B.Cu at (212.9, 113.3)
- added KD23: 1N4148, travis:Diode_DO-35, B.Cu at (235.6, 187.7)
- added KD24: 1N4148, travis:Diode_DO-35, B.Cu at (234.5, 149.6)
- added KD25: 1N4148, travis:Diode_DO-35, B.Cu at (233.3, 111.5)
- added KD26: 1N4148, travis:Diode_DO-35, B.Cu at (254.9, 188.3)
- added KD27: 1N4148, travis:Diode_DO-35, B.Cu at (254.4, 150.2)
- added KD28: 1N4148, travis:Diode_DO-35, B.Cu at (253.9, 112.1)
- added KD29: 1N4148, travis:Diode_DO-35, B.Cu at (274.1, 190.2)
- added KD3: 1N4148, travis:Diode_DO-35, B.Cu at (49.5, 115.3)
- added KD30: 1N4148, travis:Diode_DO-35, B.Cu at (274.2, 152.1)
- added KD31: 1N4148, travis:Diode_DO-35, B.Cu at (274.4, 114.0)
- added KD32: 1N4148, travis:Diode_DO-35, B.Cu at (293.1, 190.2)
- added KD33: 1N4148, travis:Diode_DO-35, B.Cu at (293.3, 152.1)
- added KD34: 1N4148, travis:Diode_DO-35, B.Cu at (293.5, 114.0)
- added KD35: 1N4148, travis:Diode_DO-35, B.Cu at (317.7, 152.2)
- added KD36: 1N4148, travis:Diode_DO-35, B.Cu at (312.5, 114.1)
- added KD37: 1N4148, travis:Diode_DO-35, B.Cu at (336.9, 114.2)
- added KD38: 1N4148, travis:Diode_DO-35, B.Cu at (336.9, 196.6)
- added KD39: 1N4148, travis:Diode_DO-35, B.Cu at (349.7, 182.4)
- added KD4: 1N4148, travis:Diode_DO-35, B.Cu at (69.2, 191.4)
- added KD40: 1N4148, travis:Diode_DO-35, B.Cu at (365.7, 164.8)
- added KD41: 1N4148, travis:Diode_DO-35, B.Cu at (378.5, 150.7)
- added KD42: 1N4148, travis:Diode_DO-35, B.Cu at (379.2, 114.4)
- added KD43: 1N4148, travis:Diode_DO-35, B.Cu at (398.2, 114.5)
- added KD44: 1N4148, travis:Diode_DO-35, B.Cu at (44.8, 172.5)
- added KD45: 1N4148, travis:Diode_DO-35, B.Cu at (44.4, 134.4)
- added KD46: 1N4148, travis:Diode_DO-35, B.Cu at (49.4, 96.3)
- added KD47: 1N4148, travis:Diode_DO-35, B.Cu at (69.1, 172.3)
- added KD48: 1N4148, travis:Diode_DO-35, B.Cu at (68.7, 134.2)
- added KD49: 1N4148, travis:Diode_DO-35, B.Cu at (88.6, 170.3)
- added KD5: 1N4148, travis:Diode_DO-35, B.Cu at (68.9, 153.3)
- added KD50: 1N4148, travis:Diode_DO-35, B.Cu at (88.9, 132.2)
- added KD51: 1N4148, travis:Diode_DO-35, B.Cu at (89.3, 94.1)
- added KD52: 1N4148, travis:Diode_DO-35, B.Cu at (108.1, 169.6)
- added KD53: 1N4148, travis:Diode_DO-35, B.Cu at (109.1, 131.5)
- added KD54: 1N4148, travis:Diode_DO-35, B.Cu at (110.1, 93.5)
- added KD55: 1N4148, travis:Diode_DO-35, B.Cu at (127.6, 171.3)
- added KD56: 1N4148, travis:Diode_DO-35, B.Cu at (129.3, 133.2)
- added KD57: 1N4148, travis:Diode_DO-35, B.Cu at (130.9, 95.2)
- added KD58: 1N4148, travis:Diode_DO-35, B.Cu at (146.7, 172.4)
- added KD59: 1N4148, travis:Diode_DO-35, B.Cu at (148.6, 134.4)
- added KD6: 1N4148, travis:Diode_DO-35, B.Cu at (68.6, 115.2)
- added KD60: 1N4148, travis:Diode_DO-35, B.Cu at (150.4, 96.3)
- added KD61: 1N4148, travis:Diode_DO-35, B.Cu at (196.6, 171.6)
- added KD62: 1N4148, travis:Diode_DO-35, B.Cu at (194.8, 133.5)
- added KD63: 1N4148, travis:Diode_DO-35, B.Cu at (192.9, 95.5)
- added KD64: 1N4148, travis:Diode_DO-35, B.Cu at (215.6, 170.4)
- added KD65: 1N4148, travis:Diode_DO-35, B.Cu at (213.8, 132.4)
- added KD66: 1N4148, travis:Diode_DO-35, B.Cu at (211.9, 94.3)
- added KD67: 1N4148, travis:Diode_DO-35, B.Cu at (235.1, 168.6)
- added KD68: 1N4148, travis:Diode_DO-35, B.Cu at (233.9, 130.6)
- added KD69: 1N4148, travis:Diode_DO-35, B.Cu at (232.7, 92.5)
- added KD7: 1N4148, travis:Diode_DO-35, B.Cu at (88.4, 189.4)
- added KD70: 1N4148, travis:Diode_DO-35, B.Cu at (254.6, 169.2)
- added KD71: 1N4148, travis:Diode_DO-35, B.Cu at (254.1, 131.1)
- added KD72: 1N4148, travis:Diode_DO-35, B.Cu at (253.6, 93.0)
- added KD73: 1N4148, travis:Diode_DO-35, B.Cu at (274.2, 171.1)
- added KD74: 1N4148, travis:Diode_DO-35, B.Cu at (274.3, 133.0)
- added KD75: 1N4148, travis:Diode_DO-35, B.Cu at (298.6, 171.2)
- added KD76: 1N4148, travis:Diode_DO-35, B.Cu at (293.4, 133.1)
- added KD77: 1N4148, travis:Diode_DO-35, B.Cu at (293.5, 95.0)
- added KD78: 1N4148, travis:Diode_DO-35, B.Cu at (312.4, 133.2)
- added KD79: 1N4148, travis:Diode_DO-35, B.Cu at (312.6, 95.1)
- added KD8: 1N4148, travis:Diode_DO-35, B.Cu at (88.8, 151.3)
- added KD80: 1N4148, travis:Diode_DO-35, B.Cu at (331.5, 133.3)
- added KD81: 1N4148, travis:Diode_DO-35, B.Cu at (331.6, 95.2)
- added KD82: 1N4148, travis:Diode_DO-35, B.Cu at (350.7, 95.2)
- added KD83: 1N4148, travis:Diode_DO-35, B.Cu at (322.8, 183.7)
- added KD84: 1N4148, travis:Diode_DO-35, B.Cu at (335.6, 169.6)
- added KD85: 1N4148, travis:Diode_DO-35, B.Cu at (351.6, 152.0)
- added KD86: 1N4148, travis:Diode_DO-35, B.Cu at (364.4, 137.9)
- added KD87: 1N4148, travis:Diode_DO-35, B.Cu at (379.3, 95.4)
- added KD88: 1N4148, travis:Diode_DO-35, B.Cu at (398.3, 95.4)
- added KD9: 1N4148, travis:Diode_DO-35, B.Cu at (89.1, 113.2)
- added KLED1: SK6812mini-e, travis:led_SK6812mini-e (per-key single-side), B.Cu at (41.8, 204.6)
- added KLED10: SK6812mini-e, travis:led_SK6812mini-e (per-key single-side), B.Cu at (98.8, 201.4)
- added KLED11: SK6812mini-e, travis:led_SK6812mini-e (per-key single-side), B.Cu at (99.8, 163.3)
- added KLED12: SK6812mini-e, travis:led_SK6812mini-e (per-key single-side), B.Cu at (100.7, 125.3)
- added KLED13: SK6812mini-e, travis:led_SK6812mini-e (per-key single-side), B.Cu at (119.3, 164.9)
- added KLED14: SK6812mini-e, travis:led_SK6812mini-e (per-key single-side), B.Cu at (121.0, 126.8)
- added KLED15: SK6812mini-e, travis:led_SK6812mini-e (per-key single-side), B.Cu at (135.2, 203.9)
- added KLED16: SK6812mini-e, travis:led_SK6812mini-e (per-key single-side), B.Cu at (138.5, 166.0)
- added KLED17: SK6812mini-e, travis:led_SK6812mini-e (per-key single-side), B.Cu at (140.3, 127.9)
- added KLED18: SK6812mini-e, travis:led_SK6812mini-e (per-key single-side), B.Cu at (191.1, 203.9)
- added KLED19: SK6812mini-e, travis:led_SK6812mini-e (per-key single-side), B.Cu at (187.8, 165.9)
- added KLED2: SK6812mini-e, travis:led_SK6812mini-e (per-key single-side), B.Cu at (36.2, 166.6)
- added KLED20: SK6812mini-e, travis:led_SK6812mini-e (per-key single-side), B.Cu at (186.0, 127.9)
- added KLED21: SK6812mini-e, travis:led_SK6812mini-e (per-key single-side), B.Cu at (206.8, 164.8)
- added KLED22: SK6812mini-e, travis:led_SK6812mini-e (per-key single-side), B.Cu at (205.0, 126.7)
- added KLED23: SK6812mini-e, travis:led_SK6812mini-e (per-key single-side), B.Cu at (227.5, 200.9)
- added KLED24: SK6812mini-e, travis:led_SK6812mini-e (per-key single-side), B.Cu at (226.4, 162.8)
- added KLED25: SK6812mini-e, travis:led_SK6812mini-e (per-key single-side), B.Cu at (225.2, 124.8)
- added KLED26: SK6812mini-e, travis:led_SK6812mini-e (per-key single-side), B.Cu at (246.5, 201.3)
- added KLED27: SK6812mini-e, travis:led_SK6812mini-e (per-key single-side), B.Cu at (246.0, 163.3)
- added KLED28: SK6812mini-e, travis:led_SK6812mini-e (per-key single-side), B.Cu at (245.5, 125.2)
- added KLED29: SK6812mini-e, travis:led_SK6812mini-e (per-key single-side), B.Cu at (265.5, 203.1)
- added KLED3: SK6812mini-e, travis:led_SK6812mini-e (per-key single-side), B.Cu at (41.1, 128.4)
- added KLED30: SK6812mini-e, travis:led_SK6812mini-e (per-key single-side), B.Cu at (265.7, 165.0)
- added KLED31: SK6812mini-e, travis:led_SK6812mini-e (per-key single-side), B.Cu at (265.8, 126.9)
- added KLED32: SK6812mini-e, travis:led_SK6812mini-e (per-key single-side), B.Cu at (284.5, 203.2)
- added KLED33: SK6812mini-e, travis:led_SK6812mini-e (per-key single-side), B.Cu at (284.7, 165.1)
- added KLED34: SK6812mini-e, travis:led_SK6812mini-e (per-key single-side), B.Cu at (284.9, 127.0)
- added KLED35: SK6812mini-e, travis:led_SK6812mini-e (per-key single-side), B.Cu at (309.1, 165.2)
- added KLED36: SK6812mini-e, travis:led_SK6812mini-e (per-key single-side), B.Cu at (303.9, 127.1)
- added KLED37: SK6812mini-e, travis:led_SK6812mini-e (per-key single-side), B.Cu at (328.3, 127.2)
- added KLED38: SK6812mini-e, travis:led_SK6812mini-e (per-key single-side), B.Cu at (340.8, 211.6)
- added KLED39: SK6812mini-e, travis:led_SK6812mini-e (per-key single-side), B.Cu at (353.6, 197.5)
- added KLED4: SK6812mini-e, travis:led_SK6812mini-e (per-key single-side), B.Cu at (60.8, 204.4)
- added KLED40: SK6812mini-e, travis:led_SK6812mini-e (per-key single-side), B.Cu at (369.6, 179.9)
- added KLED41: SK6812mini-e, travis:led_SK6812mini-e (per-key single-side), B.Cu at (382.4, 165.8)
- added KLED42: SK6812mini-e, travis:led_SK6812mini-e (per-key single-side), B.Cu at (370.6, 127.4)
- added KLED43: SK6812mini-e, travis:led_SK6812mini-e (per-key single-side), B.Cu at (389.6, 127.4)
- added KLED44: SK6812mini-e, travis:led_SK6812mini-e (per-key single-side), B.Cu at (36.4, 185.6)
- added KLED45: SK6812mini-e, travis:led_SK6812mini-e (per-key single-side), B.Cu at (36.0, 147.5)
- added KLED46: SK6812mini-e, travis:led_SK6812mini-e (per-key single-side), B.Cu at (41.0, 109.4)
- added KLED47: SK6812mini-e, travis:led_SK6812mini-e (per-key single-side), B.Cu at (60.7, 185.4)
- added KLED48: SK6812mini-e, travis:led_SK6812mini-e (per-key single-side), B.Cu at (60.3, 147.3)
- added KLED49: SK6812mini-e, travis:led_SK6812mini-e (per-key single-side), B.Cu at (79.9, 183.2)
- added KLED5: SK6812mini-e, travis:led_SK6812mini-e (per-key single-side), B.Cu at (60.5, 166.3)
- added KLED50: SK6812mini-e, travis:led_SK6812mini-e (per-key single-side), B.Cu at (80.3, 145.1)
- added KLED51: SK6812mini-e, travis:led_SK6812mini-e (per-key single-side), B.Cu at (80.6, 107.0)
- added KLED52: SK6812mini-e, travis:led_SK6812mini-e (per-key single-side), B.Cu at (99.3, 182.4)
- added KLED53: SK6812mini-e, travis:led_SK6812mini-e (per-key single-side), B.Cu at (100.2, 144.3)
- added KLED54: SK6812mini-e, travis:led_SK6812mini-e (per-key single-side), B.Cu at (101.2, 106.2)
- added KLED55: SK6812mini-e, travis:led_SK6812mini-e (per-key single-side), B.Cu at (118.5, 183.9)
- added KLED56: SK6812mini-e, travis:led_SK6812mini-e (per-key single-side), B.Cu at (120.2, 145.8)
- added KLED57: SK6812mini-e, travis:led_SK6812mini-e (per-key single-side), B.Cu at (121.8, 107.8)
- added KLED58: SK6812mini-e, travis:led_SK6812mini-e (per-key single-side), B.Cu at (137.6, 185.0)
- added KLED59: SK6812mini-e, travis:led_SK6812mini-e (per-key single-side), B.Cu at (139.4, 146.9)
- added KLED6: SK6812mini-e, travis:led_SK6812mini-e (per-key single-side), B.Cu at (60.2, 128.2)
- added KLED60: SK6812mini-e, travis:led_SK6812mini-e (per-key single-side), B.Cu at (141.3, 108.9)
- added KLED61: SK6812mini-e, travis:led_SK6812mini-e (per-key single-side), B.Cu at (188.7, 185.0)
- added KLED62: SK6812mini-e, travis:led_SK6812mini-e (per-key single-side), B.Cu at (186.9, 146.9)
- added KLED63: SK6812mini-e, travis:led_SK6812mini-e (per-key single-side), B.Cu at (185.0, 108.9)
- added KLED64: SK6812mini-e, travis:led_SK6812mini-e (per-key single-side), B.Cu at (207.7, 183.8)
- added KLED65: SK6812mini-e, travis:led_SK6812mini-e (per-key single-side), B.Cu at (205.9, 145.8)
- added KLED66: SK6812mini-e, travis:led_SK6812mini-e (per-key single-side), B.Cu at (204.1, 107.7)
- added KLED67: SK6812mini-e, travis:led_SK6812mini-e (per-key single-side), B.Cu at (226.9, 181.9)
- added KLED68: SK6812mini-e, travis:led_SK6812mini-e (per-key single-side), B.Cu at (225.8, 143.8)
- added KLED69: SK6812mini-e, travis:led_SK6812mini-e (per-key single-side), B.Cu at (224.6, 105.7)
- added KLED7: SK6812mini-e, travis:led_SK6812mini-e (per-key single-side), B.Cu at (79.8, 202.3)
- added KLED70: SK6812mini-e, travis:led_SK6812mini-e (per-key single-side), B.Cu at (246.3, 182.3)
- added KLED71: SK6812mini-e, travis:led_SK6812mini-e (per-key single-side), B.Cu at (245.8, 144.2)
- added KLED72: SK6812mini-e, travis:led_SK6812mini-e (per-key single-side), B.Cu at (245.3, 106.1)
- added KLED73: SK6812mini-e, travis:led_SK6812mini-e (per-key single-side), B.Cu at (265.6, 184.0)
- added KLED74: SK6812mini-e, travis:led_SK6812mini-e (per-key single-side), B.Cu at (265.7, 145.9)
- added KLED75: SK6812mini-e, travis:led_SK6812mini-e (per-key single-side), B.Cu at (290.0, 184.2)
- added KLED76: SK6812mini-e, travis:led_SK6812mini-e (per-key single-side), B.Cu at (284.8, 146.0)
- added KLED77: SK6812mini-e, travis:led_SK6812mini-e (per-key single-side), B.Cu at (285.0, 107.9)
- added KLED78: SK6812mini-e, travis:led_SK6812mini-e (per-key single-side), B.Cu at (303.8, 146.1)
- added KLED79: SK6812mini-e, travis:led_SK6812mini-e (per-key single-side), B.Cu at (304.0, 108.0)
- added KLED8: SK6812mini-e, travis:led_SK6812mini-e (per-key single-side), B.Cu at (80.1, 164.2)
- added KLED80: SK6812mini-e, travis:led_SK6812mini-e (per-key single-side), B.Cu at (322.9, 146.2)
- added KLED81: SK6812mini-e, travis:led_SK6812mini-e (per-key single-side), B.Cu at (323.1, 108.1)
- added KLED82: SK6812mini-e, travis:led_SK6812mini-e (per-key single-side), B.Cu at (342.1, 108.2)
- added KLED83: SK6812mini-e, travis:led_SK6812mini-e (per-key single-side), B.Cu at (326.7, 198.8)
- added KLED84: SK6812mini-e, travis:led_SK6812mini-e (per-key single-side), B.Cu at (339.5, 184.7)
- added KLED85: SK6812mini-e, travis:led_SK6812mini-e (per-key single-side), B.Cu at (355.5, 167.1)
- added KLED86: SK6812mini-e, travis:led_SK6812mini-e (per-key single-side), B.Cu at (368.3, 153.0)
- added KLED87: SK6812mini-e, travis:led_SK6812mini-e (per-key single-side), B.Cu at (370.7, 108.3)
- added KLED88: SK6812mini-e, travis:led_SK6812mini-e (per-key single-side), B.Cu at (389.7, 108.4)
- added KLED9: SK6812mini-e, travis:led_SK6812mini-e (per-key single-side), B.Cu at (80.4, 126.1)
- added KSW1: Kailh MX Switch Sockets, travis:MX, F.Cu at (41.7, 199.6)
- added KSW10: Kailh MX Switch Sockets, travis:MX, F.Cu at (98.9, 196.5)
- added KSW11: Kailh MX Switch Sockets, travis:MX, F.Cu at (99.9, 158.4)
- added KSW12: Kailh MX Switch Sockets, travis:MX, F.Cu at (100.9, 120.3)
- added KSW13: Kailh MX Switch Sockets, travis:MX, F.Cu at (119.6, 159.9)
- added KSW14: Kailh MX Switch Sockets, travis:MX, F.Cu at (121.2, 121.8)
- added KSW15: Kailh MX Switch Sockets, travis:MX, F.Cu at (135.4, 199.0)
- added KSW16: Kailh MX Switch Sockets, travis:MX, F.Cu at (138.7, 161.0)
- added KSW17: Kailh MX Switch Sockets, travis:MX, F.Cu at (140.6, 122.9)
- added KSW18: Kailh MX Switch Sockets, travis:MX, F.Cu at (190.9, 199.0)
- added KSW19: Kailh MX Switch Sockets, travis:MX, F.Cu at (187.5, 161.0)
- added KSW2: Kailh MX Switch Sockets, travis:MX, F.Cu at (36.1, 161.6)
- added KSW20: Kailh MX Switch Sockets, travis:MX, F.Cu at (185.7, 122.9)
- added KSW21: Kailh MX Switch Sockets, travis:MX, F.Cu at (206.6, 159.8)
- added KSW22: Kailh MX Switch Sockets, travis:MX, F.Cu at (204.7, 121.8)
- added KSW23: Kailh MX Switch Sockets, travis:MX, F.Cu at (227.4, 196.0)
- added KSW24: Kailh MX Switch Sockets, travis:MX, F.Cu at (226.2, 157.9)
- added KSW25: Kailh MX Switch Sockets, travis:MX, F.Cu at (225.0, 119.8)
- added KSW26: Kailh MX Switch Sockets, travis:MX, F.Cu at (246.4, 196.4)
- added KSW27: Kailh MX Switch Sockets, travis:MX, F.Cu at (245.9, 158.3)
- added KSW28: Kailh MX Switch Sockets, travis:MX, F.Cu at (245.4, 120.2)
- added KSW29: Kailh MX Switch Sockets, travis:MX, F.Cu at (265.5, 198.1)
- added KSW3: Kailh MX Switch Sockets, travis:MX, F.Cu at (41.1, 123.4)
- added KSW30: Kailh MX Switch Sockets, travis:MX, F.Cu at (265.7, 160.0)
- added KSW31: Kailh MX Switch Sockets, travis:MX, F.Cu at (265.8, 121.9)
- added KSW32: Kailh MX Switch Sockets, travis:MX, F.Cu at (284.6, 198.2)
- added KSW33: Kailh MX Switch Sockets, travis:MX, F.Cu at (284.7, 160.1)
- added KSW34: Kailh MX Switch Sockets, travis:MX, F.Cu at (284.9, 122.0)
- added KSW35: Kailh MX Switch Sockets, travis:MX, F.Cu at (309.1, 160.2)
- added KSW36: Kailh MX Switch Sockets, travis:MX, F.Cu at (303.9, 122.1)
- added KSW37: Kailh MX Switch Sockets, travis:MX, F.Cu at (328.4, 122.2)
- added KSW38: Kailh MX Switch Sockets, travis:MX, F.Cu at (337.1, 208.3)
- added KSW39: Kailh MX Switch Sockets, travis:MX, F.Cu at (349.9, 194.2)
- added KSW4: Kailh MX Switch Sockets, travis:MX, F.Cu at (60.8, 199.5)
- added KSW40: Kailh MX Switch Sockets, travis:MX, F.Cu at (365.9, 176.5)
- added KSW41: Kailh MX Switch Sockets, travis:MX, F.Cu at (378.7, 162.4)
- added KSW42: Kailh MX Switch Sockets, travis:MX, F.Cu at (370.6, 122.4)
- added KSW43: Kailh MX Switch Sockets, travis:MX, F.Cu at (389.7, 122.5)
- added KSW44: Kailh MX Switch Sockets, travis:MX, F.Cu at (36.3, 180.6)
- added KSW45: Kailh MX Switch Sockets, travis:MX, F.Cu at (36.0, 142.5)
- added KSW46: Kailh MX Switch Sockets, travis:MX, F.Cu at (40.9, 104.4)
- added KSW47: Kailh MX Switch Sockets, travis:MX, F.Cu at (60.6, 180.4)
- added KSW48: Kailh MX Switch Sockets, travis:MX, F.Cu at (60.3, 142.3)
- added KSW49: Kailh MX Switch Sockets, travis:MX, F.Cu at (80.0, 178.3)
- added KSW5: Kailh MX Switch Sockets, travis:MX, F.Cu at (60.5, 161.4)
- added KSW50: Kailh MX Switch Sockets, travis:MX, F.Cu at (80.3, 140.2)
- added KSW51: Kailh MX Switch Sockets, travis:MX, F.Cu at (80.7, 102.1)
- added KSW52: Kailh MX Switch Sockets, travis:MX, F.Cu at (99.4, 177.4)
- added KSW53: Kailh MX Switch Sockets, travis:MX, F.Cu at (100.4, 139.3)
- added KSW54: Kailh MX Switch Sockets, travis:MX, F.Cu at (101.4, 101.3)
- added KSW55: Kailh MX Switch Sockets, travis:MX, F.Cu at (118.7, 178.9)
- added KSW56: Kailh MX Switch Sockets, travis:MX, F.Cu at (120.4, 140.9)
- added KSW57: Kailh MX Switch Sockets, travis:MX, F.Cu at (122.1, 102.8)
- added KSW58: Kailh MX Switch Sockets, travis:MX, F.Cu at (137.8, 180.0)
- added KSW59: Kailh MX Switch Sockets, travis:MX, F.Cu at (139.7, 142.0)
- added KSW6: Kailh MX Switch Sockets, travis:MX, F.Cu at (60.1, 123.3)
- added KSW60: Kailh MX Switch Sockets, travis:MX, F.Cu at (141.5, 103.9)
- added KSW61: Kailh MX Switch Sockets, travis:MX, F.Cu at (188.5, 180.0)
- added KSW62: Kailh MX Switch Sockets, travis:MX, F.Cu at (186.6, 142.0)
- added KSW63: Kailh MX Switch Sockets, travis:MX, F.Cu at (184.8, 103.9)
- added KSW64: Kailh MX Switch Sockets, travis:MX, F.Cu at (207.5, 178.9)
- added KSW65: Kailh MX Switch Sockets, travis:MX, F.Cu at (205.6, 140.8)
- added KSW66: Kailh MX Switch Sockets, travis:MX, F.Cu at (203.8, 102.7)
- added KSW67: Kailh MX Switch Sockets, travis:MX, F.Cu at (226.8, 176.9)
- added KSW68: Kailh MX Switch Sockets, travis:MX, F.Cu at (225.6, 138.8)
- added KSW69: Kailh MX Switch Sockets, travis:MX, F.Cu at (224.5, 100.8)
- added KSW7: Kailh MX Switch Sockets, travis:MX, F.Cu at (79.8, 197.3)
- added KSW70: Kailh MX Switch Sockets, travis:MX, F.Cu at (246.2, 177.3)
- added KSW71: Kailh MX Switch Sockets, travis:MX, F.Cu at (245.7, 139.2)
- added KSW72: Kailh MX Switch Sockets, travis:MX, F.Cu at (245.2, 101.1)
- added KSW73: Kailh MX Switch Sockets, travis:MX, F.Cu at (265.6, 179.1)
- added KSW74: Kailh MX Switch Sockets, travis:MX, F.Cu at (265.8, 141.0)
- added KSW75: Kailh MX Switch Sockets, travis:MX, F.Cu at (290.0, 179.2)
- added KSW76: Kailh MX Switch Sockets, travis:MX, F.Cu at (284.8, 141.1)
- added KSW77: Kailh MX Switch Sockets, travis:MX, F.Cu at (285.0, 103.0)
- added KSW78: Kailh MX Switch Sockets, travis:MX, F.Cu at (303.9, 141.2)
- added KSW79: Kailh MX Switch Sockets, travis:MX, F.Cu at (304.0, 103.1)
- added KSW8: Kailh MX Switch Sockets, travis:MX, F.Cu at (80.2, 159.2)
- added KSW80: Kailh MX Switch Sockets, travis:MX, F.Cu at (322.9, 141.2)
- added KSW81: Kailh MX Switch Sockets, travis:MX, F.Cu at (323.1, 103.1)
- added KSW82: Kailh MX Switch Sockets, travis:MX, F.Cu at (342.1, 103.2)
- added KSW83: Kailh MX Switch Sockets, travis:MX, F.Cu at (323.0, 195.4)
- added KSW84: Kailh MX Switch Sockets, travis:MX, F.Cu at (335.8, 181.3)
- added KSW85: Kailh MX Switch Sockets, travis:MX, F.Cu at (351.8, 163.7)
- added KSW86: Kailh MX Switch Sockets, travis:MX, F.Cu at (364.6, 149.6)
- added KSW87: Kailh MX Switch Sockets, travis:MX, F.Cu at (370.7, 103.3)
- added KSW88: Kailh MX Switch Sockets, travis:MX, F.Cu at (389.8, 103.4)
- added KSW9: Kailh MX Switch Sockets, travis:MX, F.Cu at (80.5, 121.1)
Routing:
- net RAW: track 402.2 -> 2359.3 mm
- net row3: track 0.00 -> 440.6 mm, vias 0 -> 12
- net row0: track 0.00 -> 408.7 mm
- net row5: track 0.00 -> 399.6 mm, vias 0 -> 9
- net row4: track 0.00 -> 389.4 mm, vias 0 -> 11
- net row2: track 0.00 -> 389.3 mm, vias 0 -> 13
- net row1: track 0.00 -> 372.5 mm, vias 0 -> 15
- net col15: track 0.00 -> 259.3 mm
- net col4: track 0.00 -> 240.8 mm, vias 0 -> 2
- net col14: track 0.00 -> 226.1 mm
- net col2: track 0.00 -> 215.1 mm, vias 0 -> 2
- net col3: track 0.00 -> 193.7 mm, vias 0 -> 2
- net col0: track 0.00 -> 173.7 mm
- net col8: track 0.00 -> 149.8 mm
- net col5: track 0.00 -> 139.9 mm
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Other:
- board text added: "KC1"
- board text added: "KC10"
- board text added: "KC11"
- board text added: "KC12"
- board text added: "KC13"
- board text added: "KC14"
- board text added: "KC15"
- board text added: "KC16"
- board text added: "KC17"
- board text added: "KC18"
- board text added: "KC19"
- board text added: "KC2"
- board text added: "KC20"
- board text added: "KC21"
- board text added: "KC22"
- board text added: "KC23"
- board text added: "KC24"
- board text added: "KC25"
- board text added: "KC26"
- board text added: "KC27"
- board text added: "KC28"
- board text added: "KC29"
- board text added: "KC3"
- board text added: "KC30"
- board text added: "KC31"
- board text added: "KC32"
- board text added: "KC33"
- board text added: "KC34"
- board text added: "KC35"
- board text added: "KC36"
- board text added: "KC37"
- board text added: "KC38"
- board text added: "KC39"
- board text added: "KC4"
- board text added: "KC40"
- board text added: "KC41"
- board text added: "KC42"
- board text added: "KC43"
- board text added: "KC44"
- board text added: "KC45"
- board text added: "KC46"
- board text added: "KC47"
- board text added: "KC48"
- board text added: "KC49"
- board text added: "KC5"
- board text added: "KC50"
- board text added: "KC51"
- board text added: "KC52"
- board text added: "KC53"
- board text added: "KC54"
- board text added: "KC55"
- board text added: "KC56"
- board text added: "KC57"
- board text added: "KC58"
- board text added: "KC59"
- board text added: "KC6"
- board text added: "KC60"
- board text added: "KC61"
- board text added: "KC62"
- board text added: "KC63"
- board text added: "KC64"
- board text added: "KC65"
- board text added: "KC66"
- board text added: "KC67"
- board text added: "KC68"
- board text added: "KC69"
- board text added: "KC7"
- board text added: "KC70"
- board text added: "KC71"
- board text added: "KC72"
- board text added: "KC73"
- board text added: "KC74"
- board text added: "KC75"
- board text added: "KC76"
- board text added: "KC77"
- board text added: "KC78"
- board text added: "KC79"
- board text added: "KC8"
- board text added: "KC80"
- board text added: "KC81"
- board text added: "KC82"
- board text added: "KC83"
- board text added: "KC84"
- board text added: "KC85"
- board text added: "KC86"
- board text added: "KC87"
- board text added: "KC88"
- board text added: "KC9"
- board text added: "KD1"
- board text added: "KD10"
- board text added: "KD11"
- board text added: "KD12"
- board text added: "KD13"
- board text added: "KD14"
- board text added: "KD15"
- board text added: "KD16"
- board text added: "KD17"
- board text added: "KD18"
- board text added: "KD19"
- board text added: "KD2"
- board text added: "KD20"
- board text added: "KD21"
- board text added: "KD22"
- board text added: "KD23"
- board text added: "KD24"
- board text added: "KD25"
- board text added: "KD26"
- board text added: "KD27"
- board text added: "KD28"
- board text added: "KD29"
- board text added: "KD3"
- board text added: "KD30"
- board text added: "KD31"
- board text added: "KD32"
- board text added: "KD33"
- board text added: "KD34"
- board text added: "KD35"
- board text added: "KD36"
- board text added: "KD37"
- board text added: "KD38"
- board text added: "KD39"
- board text added: "KD4"
- board text added: "KD40"
- board text added: "KD41"
- board text added: "KD42"
- board text added: "KD43"
- board text added: "KD44"
- board text added: "KD45"
- board text added: "KD46"
- board text added: "KD47"
- board text added: "KD48"
- board text added: "KD49"
- board text added: "KD5"
- board text added: "KD50"
- board text added: "KD51"
- board text added: "KD52"
- board text added: "KD53"
- board text added: "KD54"
- board text added: "KD55"
- board text added: "KD56"
- board text added: "KD57"
- board text added: "KD58"
- board text added: "KD59"
- board text added: "KD6"
- board text added: "KD60"
- board text added: "KD61"
- board text added: "KD62"
- board text added: "KD63"
- board text added: "KD64"
- board text added: "KD65"
- board text added: "KD66"
- board text added: "KD67"
- board text added: "KD68"
- board text added: "KD69"
- board text added: "KD7"
- board text added: "KD70"
- board text added: "KD71"
- board text added: "KD72"
- board text added: "KD73"
- board text added: "KD74"
- board text added: "KD75"
- board text added: "KD76"
- board text added: "KD77"
- board text added: "KD78"
- board text added: "KD79"
- board text added: "KD8"
- board text added: "KD80"
- board text added: "KD81"
- board text added: "KD82"
- board text added: "KD83"
- board text added: "KD84"
- board text added: "KD85"
- board text added: "KD86"
- board text added: "KD87"
- board text added: "KD88"
- board text added: "KD9"
- board text removed: "C1"
- board text removed: "C10"
- board text removed: "C11"
- board text removed: "C12"
- board text removed: "C13"
- board text removed: "C14"
- board text removed: "C15"
- board text removed: "C16"
- board text removed: "C17"
- board text removed: "C18"
- board text removed: "C19"
- board text removed: "C2"
- board text removed: "C20"
- board text removed: "C21"
- board text removed: "C22"
- board text removed: "C23"
- board text removed: "C24"
- board text removed: "C25"
- board text removed: "C26"
- board text removed: "C27"
- board text removed: "C28"
- board text removed: "C29"
- board text removed: "C3"
- board text removed: "C30"
- board text removed: "C31"
- board text removed: "C32"
- board text removed: "C33"
- board text removed: "C34"
- board text removed: "C35"
- board text removed: "C36"
- board text removed: "C37"
- board text removed: "C38"
- board text removed: "C39"
- board text removed: "C4"
- board text removed: "C40"
- board text removed: "C41"
- board text removed: "C42"
- board text removed: "C43"
- board text removed: "C44"
- board text removed: "C45"
- board text removed: "C46"
- board text removed: "C47"
- board text removed: "C48"
- board text removed: "C49"
- board text removed: "C5"
- board text removed: "C50"
- board text removed: "C51"
- board text removed: "C52"
- board text removed: "C53"
- board text removed: "C54"
- board text removed: "C55"
- board text removed: "C56"
- board text removed: "C57"
- board text removed: "C58"
- board text removed: "C59"
- board text removed: "C6"
- board text removed: "C60"
- board text removed: "C61"
- board text removed: "C62"
- board text removed: "C63"
- board text removed: "C64"
- board text removed: "C65"
- board text removed: "C66"
- board text removed: "C67"
- board text removed: "C68"
- board text removed: "C69"
- board text removed: "C7"
- board text removed: "C70"
- board text removed: "C71"
- board text removed: "C72"
- board text removed: "C73"
- board text removed: "C74"
- board text removed: "C75"
- board text removed: "C76"
- board text removed: "C77"
- board text removed: "C78"
- board text removed: "C79"
- board text removed: "C8"
- board text removed: "C80"
- board text removed: "C81"
- board text removed: "C82"
- board text removed: "C83"
- board text removed: "C84"
- board text removed: "C85"
- board text removed: "C86"
- board text removed: "C87"
- board text removed: "C88"
- board text removed: "C9"
- board text removed: "D1"
- board text removed: "D10"
- board text removed: "D11"
- board text removed: "D12"
- board text removed: "D13"
- board text removed: "D14"
- board text removed: "D15"
- board text removed: "D16"
- board text removed: "D17"
- board text removed: "D18"
- board text removed: "D19"
- board text removed: "D2"
- board text removed: "D20"
- board text removed: "D21"
- board text removed: "D22"
- board text removed: "D23"
- board text removed: "D24"
- board text removed: "D25"
- board text removed: "D26"
- board text removed: "D27"
- board text removed: "D28"
- board text removed: "D29"
- board text removed: "D3"
- board text removed: "D30"
- board text removed: "D31"
- board text removed: "D32"
- board text removed: "D33"
- board text removed: "D34"
- board text removed: "D35"
- board text removed: "D36"
- board text removed: "D37"
- board text removed: "D38"
- board text removed: "D39"
- board text removed: "D4"
- board text removed: "D40"
- board text removed: "D41"
- board text removed: "D42"
- board text removed: "D43"
- board text removed: "D44"
- board text removed: "D45"
- board text removed: "D46"
- board text removed: "D47"
- board text removed: "D48"
- board text removed: "D49"
- board text removed: "D5"
- board text removed: "D50"
- board text removed: "D51"
- board text removed: "D52"
- board text removed: "D53"
- board text removed: "D54"
- board text removed: "D55"
- board text removed: "D56"
- board text removed: "D57"
- board text removed: "D58"
- board text removed: "D59"
- board text removed: "D6"
- board text removed: "D60"
- board text removed: "D61"
- board text removed: "D62"
- board text removed: "D63"
- board text removed: "D64"
- board text removed: "D65"
- board text removed: "D66"
- board text removed: "D67"
- board text removed: "D68"
- board text removed: "D69"
- board text removed: "D7"
- board text removed: "D70"
- board text removed: "D71"
- board text removed: "D72"
- board text removed: "D73"
- board text removed: "D74"
- board text removed: "D75"
- board text removed: "D76"
- board text removed: "D77"
- board text removed: "D78"
- board text removed: "D79"
- board text removed: "D8"
- board text removed: "D80"
- board text removed: "D81"
- board text removed: "D82"
- board text removed: "D83"
- board text removed: "D84"
- board text removed: "D85"
- board text removed: "D86"
- board text removed: "D87"
- board text removed: "D88"
- board text removed: "D9"
