File: output/pcbs/travis_erg2024.kicad_pcb (KiCad board)
At the start: 2 copper layers, 393.3 x 146.1 mm, 380 parts, among them SW1 SW_PUSH_6mm_H4.3mm

Commit message: stab adjust
Parts:
- moved STAB2u1 0.62 mm to (132.5, 175.3), turned to 177.25 degrees
- moved STAB3u1 0.62 mm to (132.6, 174.1)
- moved STAB2u2 0.62 mm to (191.2, 175.6), turned to 182.25 degrees
- moved STAB3u2 0.62 mm to (191.1, 174.3)
Changed lines of the file:
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@@
     (descr "MX PCB Stabilizer 2.00u 2.25u 2.50u 2.75u")
     (tags "MX Keyboard Stabilizer 2.00u 2.25u 2.50u 2.75u Cutout")
-    (at 132.5415574 174.6982491 -2.75)
+    (at 132.511811 175.3175351 177.25)
     (attr virtual)
     (fp_text reference "STAB2u1" (at 0 -2) (layer F.SilkS) hide
@@
     (descr "MX PCB Stabilizer 3.00u")
     (tags "MX Keyboard Stabilizer 3.00u Cutout")
-    (at 132.5415574 174.6982491 -2.75)
+    (at 132.57130379999998 174.0789631 -2.75)
     (attr virtual)
     (fp_text reference "STAB3u1" (at 0 -2) (layer F.SilkS) hide
@@
     (descr "MX PCB Stabilizer 2.00u 2.25u 2.50u 2.75u")
     (tags "MX Keyboard Stabilizer 2.00u 2.25u 2.50u 2.75u Cutout")
-    (at 191.1486452 174.9627056 2.25)
+    (at 191.1729863 175.58222759999998 182.25)
     (attr virtual)
     (fp_text reference "STAB2u2" (at 0 -2) (layer F.SilkS) hide
@@
     (descr "MX PCB Stabilizer 3.00u")
     (tags "MX Keyboard Stabilizer 3.00u Cutout")
-    (at 191.1486452 174.9627056 2.25)
+    (at 191.12430410000002 174.3431836 2.25)
     (attr virtual)
     (fp_text reference "STAB3u2" (at 0 -2) (layer F.SilkS) hide

Commit message: splay adjust
Parts:
- moved HOLE6 2.05 mm to (402.1, 69.1), turned to -1.5 degrees
- moved D88 2.01 mm to (402.9, 74.7), turned to 268.5 degrees
- moved S88 1.85 mm to (394.2, 82.5), turned to -1.5 degrees
- moved D43 1.85 mm to (402.4, 93.7), turned to 268.5 degrees
- moved D87 1.83 mm to (383.9, 74.2), turned to 268.5 degrees
- moved LED88 1.81 mm to (394.0, 87.4), turned to 178.5 degrees
- moved C88 1.76 mm to (391.5, 90.7), turned to -1.5 degrees
- moved S43 1.70 mm to (393.7, 101.5), turned to -1.5 degrees
- moved S87 1.68 mm to (375.1, 82.0), turned to -1.5 degrees
- moved C43 1.66 mm to (396.0, 109.9), turned to 178.5 degrees
- moved LED43 1.66 mm to (393.5, 106.5), turned to -1.5 degrees
- moved D42 1.65 mm to (383.4, 93.2), turned to 268.5 degrees
- moved LED87 1.63 mm to (375.0, 86.9), turned to 178.5 degrees
- moved D82 1.60 mm to (355.3, 73.4), turned to 268.5 degrees
- moved C87 1.58 mm to (372.4, 90.2), turned to -1.5 degrees
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Other:
- board size 393.3 x 146.1 mm -> 394.8 x 146.1 mm

Commit message: adjusting splay
Parts:
- removed the C1 at (39.3, 183.1)
- removed the C1 at (163.8, 75.7)
- removed the C2 at (33.9, 145.1)
- removed the C2 at (57.9, 64.6)
- removed the C3 at (39.0, 106.9)
- removed the C3 at (270.9, 64.7)
- removed the D1 at (45.3, 166.8)
- removed the D1 at (154.0, 102.7)
- removed the D2 at (39.8, 128.7)
- removed the D2 at (155.7, 161.7)
- removed STAB3u1, STAB3u2: Stabilizer_MX_3.00u, Stabilizer_MX_3.00u
- added C1: 104, C_Disc_D4.7mm_W2.5mm_P5.00mm, B.Cu at (40.1, 183.0)
- added C1: C_Radial_D6.3mm_H11.0mm_P2.50mm, C_Radial_D6.3mm_H11.0mm_P2.50mm, B.Cu at (160.2, 74.9)
- added C2: 104, C_Disc_D4.7mm_W2.5mm_P5.00mm, B.Cu at (34.5, 144.9)
- added C2: C_Disc_D3.8mm_W2.6mm_P2.50mm, C_Disc_D3.8mm_W2.6mm_P2.50mm, F.Cu at (57.8, 64.3)
- added C3: 104, C_Disc_D4.7mm_W2.5mm_P5.00mm, B.Cu at (39.4, 106.8)
- added C3: C_Disc_D3.8mm_W2.6mm_P2.50mm, C_Disc_D3.8mm_W2.6mm_P2.50mm, F.Cu at (262.1, 63.2)
- added D1: 1N4148, Diode_DO-35, B.Cu at (46.0, 166.6)
- added D1: 1N4148, Diode_DO-35, B.Cu at (147.9, 103.0)
- added D2: 1N4148, Diode_DO-35, B.Cu at (40.4, 128.5)
- added D2: 1N4148, Diode_DO-35, B.Cu at (149.4, 160.0)
- moved HOLE6 9.86 mm to (393.1, 65.0), turned to -0.25 degrees
- moved D88 9.76 mm to (394.1, 70.5), turned to 269.75 degrees
- moved D87 9.60 mm to (375.0, 70.4), turned to 269.75 degrees
- moved S88 9.53 mm to (385.5, 78.5), turned to -0.25 degrees
- moved LED88 9.43 mm to (385.5, 83.4), turned to 179.75 degrees
- moved D43 9.39 mm to (394.0, 89.5), turned to 269.75 degrees
- moved D82 9.38 mm to (346.5, 70.3), turned to 269.75 degrees
- moved S87 9.36 mm to (366.5, 78.4), turned to -0.25 degrees
- moved C88 9.34 mm to (383.0, 86.8), turned to -0.25 degrees
- moved LED87 9.26 mm to (366.5, 83.3), turned to 179.75 degrees
- moved D81 9.25 mm to (327.4, 70.2), turned to 269.75 degrees
- moved D42 9.21 mm to (375.0, 89.4), turned to 269.75 degrees
- moved C87 9.18 mm to (363.9, 86.7), turned to -0.25 degrees
- moved S82 9.15 mm to (337.9, 78.3), turned to -0.25 degrees
- moved S43 9.15 mm to (385.5, 97.5), turned to -0.25 degrees
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Other:
- board size 394.8 x 146.1 mm -> 385.3 x 144.8 mm

Commit message: footprint updates
Parts:
- removed the C1 at (40.1, 183.0)
- removed the C1 at (160.2, 74.9)
- removed the C2 at (34.5, 144.9)
- removed the C2 at (57.8, 64.3)
- removed the C3 at (39.4, 106.8)
- removed the C3 at (262.1, 63.2)
- removed the D1 at (46.0, 166.6)
- removed the D1 at (147.9, 103.0)
- removed the D2 at (40.4, 128.5)
- removed the D2 at (149.4, 160.0)
- added C1: 104, travis:C_Disc_D4.7mm_W2.5mm_P5.00mm, B.Cu at (40.1, 183.0)
- added C1: C_Radial_D6.3mm_H11.0mm_P2.50mm, travis:C_Radial_D6.3mm_H11.0mm_P2.50mm, B.Cu at (160.2, 70.9)
- added C2: 104, travis:C_Disc_D4.7mm_W2.5mm_P5.00mm, B.Cu at (34.5, 144.9)
- added C2: C_Disc_D3.8mm_W2.6mm_P2.50mm, travis:C_Disc_D3.8mm_W2.6mm_P2.50mm, F.Cu at (57.8, 64.3)
- added C3: 104, travis:C_Disc_D4.7mm_W2.5mm_P5.00mm, B.Cu at (39.4, 106.8)
- added C3: C_Disc_D3.8mm_W2.6mm_P2.50mm, travis:C_Disc_D3.8mm_W2.6mm_P2.50mm, F.Cu at (262.1, 63.2)
- added D1: 1N4148, travis:Diode_DO-35, B.Cu at (46.0, 166.6)
- added D1: 1N4148, travis:Diode_DO-35, B.Cu at (147.9, 103.0)
- added D2: 1N4148, travis:Diode_DO-35, B.Cu at (40.4, 128.5)
- added D2: 1N4148, travis:Diode_DO-35, B.Cu at (149.4, 160.0)
- C10, C11, C12, C13, C14, C15, C16, C17, C18, C19, C20, C21, C22, C23, C24, C25, C26, C27, C28, C29, C30, C31, C32, C33, C34, C35, C36, C37, C38, C39, C4, C40, C41, C42, C43, C44, C45, C46, C47, C48, C49, C5, C50, C51, C52, C53, C54, C55, C56, C57, C58, C59, C6, C60, C61, C62, C63, C64, C65, C66, C67, C68, C69, C7, C70, C71, C72, C73, C74, C75, C76, C77, C78, C79, C8, C80, C81, C82, C83, C84, C85, C86, C87, C88, C9: footprint C_Disc_D4.7mm_W2.5mm_P5.00mm -> travis:C_Disc_D4.7mm_W2.5mm_P5.00mm
- D10, D11, D12, D13, D14, D15, D16, D17, D18, D19, D20, D21, D22, D23, D24, D25, D26, D27, D28, D29, D3, D30, D31, D32, D33, D34, D35, D36, D37, D38, D39, D4, D40, D41, D42, D43, D44, D45, D46, D47, D48, D49, D5, D50, D51, D52, D53, D54, D55, D56, D57, D58, D59, D6, D60, D61, D62, D63, D64, D65, D66, D67, D68, D69, D7, D70, D71, D72, D73, D74, D75, D76, D77, D78, D79, D8, D80, D81, D82, D83, D84, D85, D86, D87, D88, D9: footprint Diode_DO-35 -> travis:Diode_DO-35
- DIP1, DIP2: footprint DIP-16_W7.62mm_Socket -> travis:DIP-16_W7.62mm_Socket
- HOLE1, HOLE2, HOLE3, HOLE4, HOLE5, HOLE6, HOLE7, HOLE8, HOLE9: footprint MountingHole_2.2mm_M2_Pad_Via -> travis:MountingHole_2.2mm_M2_Pad_Via
- LED1, LED10, LED11, LED12, LED13, LED14, LED15, LED16, LED17, LED18, LED19, LED2, LED20, LED21, LED22, LED23, LED24, LED25, LED26, LED27, LED28, LED29, LED3, LED30, LED31, LED32, LED33, LED34, LED35, LED36, LED37, LED38, LED39, LED4, LED40, LED41, LED42, LED43, LED44, LED45, LED46, LED47, LED48, LED49, LED5, LED50, LED51, LED52, LED53, LED54, LED55, LED56, LED57, LED58, LED59, LED6, LED60, LED61, LED62, LED63, LED64, LED65, LED66, LED67, LED68, LED69, LED7, LED70, LED71, LED72, LED73, LED74, LED75, LED76, LED77, LED78, LED79, LED8, LED80, LED81, LED82, LED83, LED84, LED85, LED86, LED87, LED88, LED9: footprint ceoloide:led_SK6812mini-e (per-key single-side) -> travis:led_SK6812mini-e (per-key single-side)
- LOGO1: footprint ergogen -> travis:ergogen
- LOGO2: footprint travis -> travis:travis
- R1: footprint R_Axial_DIN0207_L6.3mm_D2.5mm_P10.16mm_Horizontal -> travis:R_Axial_DIN0207_L6.3mm_D2.5mm_P10.16mm_Horizontal
- S1, S10, S11, S12, S13, S14, S15, S16, S17, S18, S19, S2, S20, S21, S22, S23, S24, S25, S26, S27, S28, S29, S3, S30, S31, S32, S33, S34, S35, S36, S37, S38, S39, S4, S40, S41, S42, S43, S44, S45, S46, S47, S48, S49, S5, S50, S51, S52, S53, S54, S55, S56, S57, S58, S59, S6, S60, S61, S62, S63, S64, S65, S66, S67, S68, S69, S7, S70, S71, S72, S73, S74, S75, S76, S77, S78, S79, S8, S80, S81, S82, S83, S84, S85, S86, S87, S88, S9: footprint MX -> travis:MX
- STAB2u1, STAB2u2: footprint Stabilizer_MX_2.00u -> travis:Stabilizer_MX_2.00u
- SW1: footprint SW_PUSH_6mm_H4.3mm -> travis:SW_PUSH_6mm_H4.3mm
- SYM1: footprint KiCad-Logo_5mm_Copper -> travis:KiCad-Logo_5mm_Copper
Other:
- board text added: "arrows_left_bottom col15 row5"
- board text added: "arrows_left_top col14 row5"
- board text added: "arrows_right_bottom col15 row4"
- board text added: "arrows_right_top col14 row4"
- board text added: "matrixl_index_bottom col4 row4"
- board text added: "matrixl_index_func col4 row0"
- board text added: "matrixl_index_home col4 row3"
- board text added: "matrixl_index_num col4 row1"
- board text added: "matrixl_index_top col4 row2"
- board text added: "matrixl_inner_bottom col5 row4"
- board text added: "matrixl_inner_func col5 row0"
- board text added: "matrixl_inner_home col5 row3"
- board text added: "matrixl_inner_mod col5 row5"
- board text added: "matrixl_inner_num col5 row1"
- board text added: "matrixl_inner_top col5 row2"
- board text added: "matrixl_middle_bottom col3 row4"
- board text added: "matrixl_middle_func col3 row0"
- board text added: "matrixl_middle_home col3 row3"
- board text added: "matrixl_middle_mod col3 row5"
- board text added: "matrixl_middle_num col3 row1"
- board text added: "matrixl_middle_top col3 row2"
- board text added: "matrixl_outer_bottom col0 row4"
- board text added: "matrixl_outer_func col0 row0"
- board text added: "matrixl_outer_home col0 row3"
- board text added: "matrixl_outer_mod col0 row5"
- board text added: "matrixl_outer_num col0 row1"
- board text added: "matrixl_outer_top col0 row2"
- board text added: "matrixl_pinky_bottom col1 row4"
- board text added: "matrixl_pinky_home col1 row3"
- board text added: "matrixl_pinky_mod col1 row5"
- board text added: "matrixl_pinky_num col1 row1"
- board text added: "matrixl_pinky_top col1 row2"
- board text added: "matrixl_ring_bottom col2 row4"
- board text added: "matrixl_ring_func col2 row0"
- board text added: "matrixl_ring_home col2 row3"
- board text added: "matrixl_ring_mod col2 row5"
- board text added: "matrixl_ring_num col2 row1"
- board text added: "matrixl_ring_top col2 row2"
- board text added: "matrixr_index_bottom col7 row4"
- board text added: "matrixr_index_func col7 row0"
- board text added: "matrixr_index_home col7 row3"
- board text added: "matrixr_index_num col7 row1"
- board text added: "matrixr_index_top col7 row2"
- board text added: "matrixr_inner_bottom col6 row4"
- board text added: "matrixr_inner_func col6 row0"
- board text added: "matrixr_inner_home col6 row3"
- board text added: "matrixr_inner_mod col6 row5"
- board text added: "matrixr_inner_num col6 row1"
- board text added: "matrixr_inner_top col6 row2"
- board text added: "matrixr_middle_bottom col8 row4"
- board text added: "matrixr_middle_func col8 row0"
- board text added: "matrixr_middle_home col8 row3"
- board text added: "matrixr_middle_mod col8 row5"
- board text added: "matrixr_middle_num col8 row1"
- board text added: "matrixr_middle_top col8 row2"
- board text added: "matrixr_outer2_func col12 row0"
- board text added: "matrixr_outer2_home col12 row3"
- board text added: "matrixr_outer2_num col12 row1"
- board text added: "matrixr_outer2_top col12 row2"
- board text added: "matrixr_outer3_func col13 row0"
- board text added: "matrixr_outer3_num col13 row1"
- board text added: "matrixr_outer3_top col13 row2"
- board text added: "matrixr_outer4_func col13 row3"
- board text added: "matrixr_outer_bottom col11 row4"
- board text added: "matrixr_outer_func col11 row0"
- board text added: "matrixr_outer_home col11 row3"
- board text added: "matrixr_outer_mod col11 row5"
- board text added: "matrixr_outer_num col11 row1"
- board text added: "matrixr_outer_top col11 row2"
- board text added: "matrixr_pinky_bottom col10 row4"
- board text added: "matrixr_pinky_home col10 row3"
- board text added: "matrixr_pinky_mod col10 row5"
- board text added: "matrixr_pinky_num col10 row1"
- board text added: "matrixr_pinky_top col10 row2"
- board text added: "matrixr_ring_bottom col9 row4"
- board text added: "matrixr_ring_func col9 row0"
- board text added: "matrixr_ring_home col9 row3"
- board text added: "matrixr_ring_mod col9 row5"
- board text added: "matrixr_ring_num col9 row1"
- board text added: "matrixr_ring_top col9 row2"
- board text added: "pages_left_bottom col15 row3"
- board text added: "pages_left_top col14 row3"
- board text added: "pages_right_bottom col15 row2"
- board text added: "pages_right_top col14 row2"
- board text added: "special_left_bottom col14 row1"
- board text added: "special_left_top col14 row0"
- board text added: "special_right_bottom col15 row1"
- board text added: "special_right_top col15 row0"

Commit message: pcb render
Parts:
- removed the C1 at (40.1, 183.0)
- removed the C1 at (160.2, 70.9)
- removed the C2 at (34.5, 144.9)
- removed the C2 at (57.8, 64.3)
- removed the C3 at (39.4, 106.8)
- removed the C3 at (262.1, 63.2)
- removed the D1 at (46.0, 166.6)
- removed the D1 at (147.9, 103.0)
- removed the D2 at (40.4, 128.5)
- removed the D2 at (149.4, 160.0)
- added C1: 104, travis:C_Disc_D4.7mm_W2.5mm_P5.00mm, B.Cu at (44.3, 207.9)
- added C1: C_Radial_D6.3mm_H11.0mm_P2.50mm, travis:C_Radial_D6.3mm_H11.0mm_P2.50mm, B.Cu at (164.4, 95.9)
- added C2: 104, travis:C_Disc_D4.7mm_W2.5mm_P5.00mm, B.Cu at (38.7, 169.9)
- added C2: C_Disc_D3.8mm_W2.6mm_P2.50mm, travis:C_Disc_D3.8mm_W2.6mm_P2.50mm, F.Cu at (62.0, 89.3)
- added C3: 104, travis:C_Disc_D4.7mm_W2.5mm_P5.00mm, B.Cu at (43.7, 131.7)
- added C3: C_Disc_D3.8mm_W2.6mm_P2.50mm, travis:C_Disc_D3.8mm_W2.6mm_P2.50mm, F.Cu at (266.3, 88.1)
- added D1: 1N4148, travis:Diode_DO-35, B.Cu at (50.2, 191.5)
- added D1: 1N4148, travis:Diode_DO-35, B.Cu at (152.1, 128.0)
- added D2: 1N4148, travis:Diode_DO-35, B.Cu at (44.6, 153.5)
- added D2: 1N4148, travis:Diode_DO-35, B.Cu at (153.6, 185.0)
- moved SW1 26.8 mm to (180.8, 87.8)
- moved C31 25.3 mm to (268.3, 130.3)
- moved D23 25.3 mm to (235.6, 187.7)
- moved D28 25.3 mm to (253.9, 112.1)
- moved LED19 25.3 mm to (187.8, 165.9)
- moved C70 25.3 mm to (243.8, 185.7)
- moved C79 25.3 mm to (301.5, 111.3)
- moved LED42 25.3 mm to (370.6, 127.4)
- moved LED53 25.3 mm to (100.2, 144.3)
- moved LED75 25.3 mm to (290.0, 184.2)
- moved LED37 25.3 mm to (328.3, 127.2)
- moved D57 25.3 mm to (130.9, 95.2)
- moved D40 25.3 mm to (365.7, 164.8)
- moved LED58 25.3 mm to (137.6, 185.0)
- moved C22 25.3 mm to (207.6, 129.9)
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Other:
- outline, holes or cut-outs redrawn

Commit message: minor label fix
Parts:
- removed the C1 at (44.3, 207.9)
- removed C10, C11, C12, C13, C14, C15, C16, C17, C18, C19, C20, C21, C22, C23, C24, C25, C26, C27, C28, C29, C30, C31, C32, C33, C34, C35, C36, C37, C38, C39, C4, C40, C41, C42, C43, C44, C45, C46, C47, C48, C49, C5, C50, C51, C52, C53, C54, C55, C56, C57, C58, C59, C6, C60, C61, C62, C63, C64, C65, C66, C67, C68, C69, C7, C70, C71, C72, C73, C74, C75, C76, C77, C78, C79, C8, C80, C81, C82, C83, C84, C85, C86, C87, C88, C9: 104, travis:C_Disc_D4.7mm_W2.5mm_P5.00mm
- removed the C2 at (38.7, 169.9)
- removed the C3 at (43.7, 131.7)
- removed the D1 at (50.2, 191.5)
- removed D10, D11, D12, D13, D14, D15, D16, D17, D18, D19, D20, D21, D22, D23, D24, D25, D26, D27, D28, D29, D3, D30, D31, D32, D33, D34, D35, D36, D37, D38, D39, D4, D40, D41, D42, D43, D44, D45, D46, D47, D48, D49, D5, D50, D51, D52, D53, D54, D55, D56, D57, D58, D59, D6, D60, D61, D62, D63, D64, D65, D66, D67, D68, D69, D7, D70, D71, D72, D73, D74, D75, D76, D77, D78, D79, D8, D80, D81, D82, D83, D84, D85, D86, D87, D88, D9: 1N4148, travis:Diode_DO-35
- removed the D2 at (44.6, 153.5)
- removed LED1, LED10, LED11, LED12, LED13, LED14, LED15, LED16, LED17, LED18, LED19, LED2, LED20, LED21, LED22, LED23, LED24, LED25, LED26, LED27, LED28, LED29, LED3, LED30, LED31, LED32, LED33, LED34, LED35, LED36, LED37, LED38, LED39, LED4, LED40, LED41, LED42, LED43, LED44, LED45, LED46, LED47, LED48, LED49, LED5, LED50, LED51, LED52, LED53, LED54, LED55, LED56, LED57, LED58, LED59, LED6, LED60, LED61, LED62, LED63, LED64, LED65, LED66, LED67, LED68, LED69, LED7, LED70, LED71, LED72, LED73, LED74, LED75, LED76, LED77, LED78, LED79, LED8, LED80, LED81, LED82, LED83, LED84, LED85, LED86, LED87, LED88, LED9: SK6812mini-e, travis:led_SK6812mini-e (per-key single-side)
- removed S1, S10, S11, S12, S13, S14, S15, S16, S17, S18, S19, S2, S20, S21, S22, S23, S24, S25, S26, S27, S28, S29, S3, S30, S31, S32, S33, S34, S35, S36, S37, S38, S39, S4, S40, S41, S42, S43, S44, S45, S46, S47, S48, S49, S5, S50, S51, S52, S53, S54, S55, S56, S57, S58, S59, S6, S60, S61, S62, S63, S64, S65, S66, S67, S68, S69, S7, S70, S71, S72, S73, S74, S75, S76, S77, S78, S79, S8, S80, S81, S82, S83, S84, S85, S86, S87, S88, S9: Kailh MX Switch Sockets, travis:MX
- added KC1: 104, travis:C_Disc_D4.7mm_W2.5mm_P5.00mm, B.Cu at (44.3, 207.9)
- added KC10: 104, travis:C_Disc_D4.7mm_W2.5mm_P5.00mm, B.Cu at (101.2, 204.8)
- added KC11: 104, travis:C_Disc_D4.7mm_W2.5mm_P5.00mm, B.Cu at (102.2, 166.8)
- added KC12: 104, travis:C_Disc_D4.7mm_W2.5mm_P5.00mm, B.Cu at (103.2, 128.7)
- added KC13: 104, travis:C_Disc_D4.7mm_W2.5mm_P5.00mm, B.Cu at (121.7, 168.3)
- added KC14: 104, travis:C_Disc_D4.7mm_W2.5mm_P5.00mm, B.Cu at (123.4, 130.2)
- added KC15: 104, travis:C_Disc_D4.7mm_W2.5mm_P5.00mm, B.Cu at (137.5, 207.4)
- added KC16: 104, travis:C_Disc_D4.7mm_W2.5mm_P5.00mm, B.Cu at (140.8, 169.4)
- added KC17: 104, travis:C_Disc_D4.7mm_W2.5mm_P5.00mm, B.Cu at (142.7, 131.4)
- added KC18: 104, travis:C_Disc_D4.7mm_W2.5mm_P5.00mm, B.Cu at (193.8, 207.1)
- added KC19: 104, travis:C_Disc_D4.7mm_W2.5mm_P5.00mm, B.Cu at (190.4, 169.2)
- added KC2: 104, travis:C_Disc_D4.7mm_W2.5mm_P5.00mm, B.Cu at (38.7, 169.9)
- added KC20: 104, travis:C_Disc_D4.7mm_W2.5mm_P5.00mm, B.Cu at (188.6, 131.1)
- added KC21: 104, travis:C_Disc_D4.7mm_W2.5mm_P5.00mm, B.Cu at (209.5, 168.0)
- added KC22: 104, travis:C_Disc_D4.7mm_W2.5mm_P5.00mm, B.Cu at (207.6, 129.9)
- added KC23: 104, travis:C_Disc_D4.7mm_W2.5mm_P5.00mm, B.Cu at (230.1, 204.2)
- added KC24: 104, travis:C_Disc_D4.7mm_W2.5mm_P5.00mm, B.Cu at (229.0, 166.1)
- added KC25: 104, travis:C_Disc_D4.7mm_W2.5mm_P5.00mm, B.Cu at (227.8, 128.0)
- added KC26: 104, travis:C_Disc_D4.7mm_W2.5mm_P5.00mm, B.Cu at (249.0, 204.7)
- added KC27: 104, travis:C_Disc_D4.7mm_W2.5mm_P5.00mm, B.Cu at (248.5, 166.6)
- added KC28: 104, travis:C_Disc_D4.7mm_W2.5mm_P5.00mm, B.Cu at (248.0, 128.5)
- added KC29: 104, travis:C_Disc_D4.7mm_W2.5mm_P5.00mm, B.Cu at (268.0, 206.5)
- added KC3: 104, travis:C_Disc_D4.7mm_W2.5mm_P5.00mm, B.Cu at (43.7, 131.7)
- added KC30: 104, travis:C_Disc_D4.7mm_W2.5mm_P5.00mm, B.Cu at (268.1, 168.4)
- added KC31: 104, travis:C_Disc_D4.7mm_W2.5mm_P5.00mm, B.Cu at (268.3, 130.3)
- added KC32: 104, travis:C_Disc_D4.7mm_W2.5mm_P5.00mm, B.Cu at (287.0, 206.5)
- added KC33: 104, travis:C_Disc_D4.7mm_W2.5mm_P5.00mm, B.Cu at (287.2, 168.4)
- added KC34: 104, travis:C_Disc_D4.7mm_W2.5mm_P5.00mm, B.Cu at (287.4, 130.3)
- added KC35: 104, travis:C_Disc_D4.7mm_W2.5mm_P5.00mm, B.Cu at (311.6, 168.5)
- added KC36: 104, travis:C_Disc_D4.7mm_W2.5mm_P5.00mm, B.Cu at (306.4, 130.4)
- added KC37: 104, travis:C_Disc_D4.7mm_W2.5mm_P5.00mm, B.Cu at (330.8, 130.5)
- added KC38: 104, travis:C_Disc_D4.7mm_W2.5mm_P5.00mm, B.Cu at (344.9, 212.0)
- added KC39: 104, travis:C_Disc_D4.7mm_W2.5mm_P5.00mm, B.Cu at (357.8, 197.9)
- added KC4: 104, travis:C_Disc_D4.7mm_W2.5mm_P5.00mm, B.Cu at (63.4, 207.8)
- added KC40: 104, travis:C_Disc_D4.7mm_W2.5mm_P5.00mm, B.Cu at (373.8, 180.3)
- added KC41: 104, travis:C_Disc_D4.7mm_W2.5mm_P5.00mm, B.Cu at (386.6, 166.2)
- added KC42: 104, travis:C_Disc_D4.7mm_W2.5mm_P5.00mm, B.Cu at (373.1, 130.7)
- added KC43: 104, travis:C_Disc_D4.7mm_W2.5mm_P5.00mm, B.Cu at (392.1, 130.8)
- added KC44: 104, travis:C_Disc_D4.7mm_W2.5mm_P5.00mm, B.Cu at (33.9, 189.0)
- added KC45: 104, travis:C_Disc_D4.7mm_W2.5mm_P5.00mm, B.Cu at (33.6, 150.9)
- added KC46: 104, travis:C_Disc_D4.7mm_W2.5mm_P5.00mm, B.Cu at (38.5, 112.7)
- added KC47: 104, travis:C_Disc_D4.7mm_W2.5mm_P5.00mm, B.Cu at (58.2, 188.7)
- added KC48: 104, travis:C_Disc_D4.7mm_W2.5mm_P5.00mm, B.Cu at (57.9, 150.7)
- added KC49: 104, travis:C_Disc_D4.7mm_W2.5mm_P5.00mm, B.Cu at (77.4, 186.5)
- added KC5: 104, travis:C_Disc_D4.7mm_W2.5mm_P5.00mm, B.Cu at (63.0, 169.7)
- added KC50: 104, travis:C_Disc_D4.7mm_W2.5mm_P5.00mm, B.Cu at (77.8, 148.4)
- added KC51: 104, travis:C_Disc_D4.7mm_W2.5mm_P5.00mm, B.Cu at (78.1, 110.3)
- added KC52: 104, travis:C_Disc_D4.7mm_W2.5mm_P5.00mm, B.Cu at (96.7, 185.7)
- added KC53: 104, travis:C_Disc_D4.7mm_W2.5mm_P5.00mm, B.Cu at (97.7, 147.6)
- added KC54: 104, travis:C_Disc_D4.7mm_W2.5mm_P5.00mm, B.Cu at (98.7, 109.5)
- added KC55: 104, travis:C_Disc_D4.7mm_W2.5mm_P5.00mm, B.Cu at (115.9, 187.1)
- added KC56: 104, travis:C_Disc_D4.7mm_W2.5mm_P5.00mm, B.Cu at (117.5, 149.1)
- added KC57: 104, travis:C_Disc_D4.7mm_W2.5mm_P5.00mm, B.Cu at (119.2, 111.0)
- added KC58: 104, travis:C_Disc_D4.7mm_W2.5mm_P5.00mm, B.Cu at (134.9, 188.2)
- added KC59: 104, travis:C_Disc_D4.7mm_W2.5mm_P5.00mm, B.Cu at (136.8, 150.1)
- added KC6: 104, travis:C_Disc_D4.7mm_W2.5mm_P5.00mm, B.Cu at (62.7, 131.6)
- added KC60: 104, travis:C_Disc_D4.7mm_W2.5mm_P5.00mm, B.Cu at (138.6, 112.1)
- added KC61: 104, travis:C_Disc_D4.7mm_W2.5mm_P5.00mm, B.Cu at (186.4, 188.4)
- added KC62: 104, travis:C_Disc_D4.7mm_W2.5mm_P5.00mm, B.Cu at (184.5, 150.4)
- added KC63: 104, travis:C_Disc_D4.7mm_W2.5mm_P5.00mm, B.Cu at (182.7, 112.3)
- added KC64: 104, travis:C_Disc_D4.7mm_W2.5mm_P5.00mm, B.Cu at (205.4, 187.3)
- added KC65: 104, travis:C_Disc_D4.7mm_W2.5mm_P5.00mm, B.Cu at (203.5, 149.2)
- added KC66: 104, travis:C_Disc_D4.7mm_W2.5mm_P5.00mm, B.Cu at (201.7, 111.2)
- added KC67: 104, travis:C_Disc_D4.7mm_W2.5mm_P5.00mm, B.Cu at (224.5, 185.3)
- added KC68: 104, travis:C_Disc_D4.7mm_W2.5mm_P5.00mm, B.Cu at (223.4, 147.2)
- added KC69: 104, travis:C_Disc_D4.7mm_W2.5mm_P5.00mm, B.Cu at (222.2, 109.1)
- added KC7: 104, travis:C_Disc_D4.7mm_W2.5mm_P5.00mm, B.Cu at (82.3, 205.6)
- added KC70: 104, travis:C_Disc_D4.7mm_W2.5mm_P5.00mm, B.Cu at (243.8, 185.7)
- added KC71: 104, travis:C_Disc_D4.7mm_W2.5mm_P5.00mm, B.Cu at (243.3, 147.6)
- added KC72: 104, travis:C_Disc_D4.7mm_W2.5mm_P5.00mm, B.Cu at (242.8, 109.5)
- added KC73: 104, travis:C_Disc_D4.7mm_W2.5mm_P5.00mm, B.Cu at (263.1, 187.4)
- added KC74: 104, travis:C_Disc_D4.7mm_W2.5mm_P5.00mm, B.Cu at (263.2, 149.3)
- added KC75: 104, travis:C_Disc_D4.7mm_W2.5mm_P5.00mm, B.Cu at (287.5, 187.5)
- added KC76: 104, travis:C_Disc_D4.7mm_W2.5mm_P5.00mm, B.Cu at (282.3, 149.4)
- added KC77: 104, travis:C_Disc_D4.7mm_W2.5mm_P5.00mm, B.Cu at (282.4, 111.3)
- added KC78: 104, travis:C_Disc_D4.7mm_W2.5mm_P5.00mm, B.Cu at (301.3, 149.4)
- added KC79: 104, travis:C_Disc_D4.7mm_W2.5mm_P5.00mm, B.Cu at (301.5, 111.3)
- added KC8: 104, travis:C_Disc_D4.7mm_W2.5mm_P5.00mm, B.Cu at (82.6, 167.5)
- added KC80: 104, travis:C_Disc_D4.7mm_W2.5mm_P5.00mm, B.Cu at (320.4, 149.5)
- added KC81: 104, travis:C_Disc_D4.7mm_W2.5mm_P5.00mm, B.Cu at (320.5, 111.4)
- added KC82: 104, travis:C_Disc_D4.7mm_W2.5mm_P5.00mm, B.Cu at (339.6, 111.5)
- added KC83: 104, travis:C_Disc_D4.7mm_W2.5mm_P5.00mm, B.Cu at (327.5, 202.9)
- added KC84: 104, travis:C_Disc_D4.7mm_W2.5mm_P5.00mm, B.Cu at (340.3, 188.8)
- added KC85: 104, travis:C_Disc_D4.7mm_W2.5mm_P5.00mm, B.Cu at (356.3, 171.2)
- added KC86: 104, travis:C_Disc_D4.7mm_W2.5mm_P5.00mm, B.Cu at (369.1, 157.1)
- added KC87: 104, travis:C_Disc_D4.7mm_W2.5mm_P5.00mm, B.Cu at (368.2, 111.6)
- added KC88: 104, travis:C_Disc_D4.7mm_W2.5mm_P5.00mm, B.Cu at (387.2, 111.7)
- added KC9: 104, travis:C_Disc_D4.7mm_W2.5mm_P5.00mm, B.Cu at (82.9, 129.4)
- added KD1: 1N4148, travis:Diode_DO-35, B.Cu at (50.2, 191.5)
- added KD10: 1N4148, travis:Diode_DO-35, B.Cu at (107.6, 188.7)
- added KD11: 1N4148, travis:Diode_DO-35, B.Cu at (108.6, 150.6)
- added KD12: 1N4148, travis:Diode_DO-35, B.Cu at (109.6, 112.5)
- added KD13: 1N4148, travis:Diode_DO-35, B.Cu at (128.4, 152.3)
- added KD14: 1N4148, travis:Diode_DO-35, B.Cu at (130.1, 114.2)
- added KD15: 1N4148, travis:Diode_DO-35, B.Cu at (144.3, 191.4)
- added KD16: 1N4148, travis:Diode_DO-35, B.Cu at (147.6, 153.4)
- added KD17: 1N4148, travis:Diode_DO-35, B.Cu at (149.5, 115.3)
- added KD18: 1N4148, travis:Diode_DO-35, B.Cu at (199.0, 190.6)
- added KD19: 1N4148, travis:Diode_DO-35, B.Cu at (195.7, 152.6)
- added KD2: 1N4148, travis:Diode_DO-35, B.Cu at (44.6, 153.5)
- added KD20: 1N4148, travis:Diode_DO-35, B.Cu at (193.8, 114.5)
- added KD21: 1N4148, travis:Diode_DO-35, B.Cu at (214.7, 151.4)
- added KD22: 1N4148, travis:Diode_DO-35, B.Cu at (212.9, 113.3)
- added KD23: 1N4148, travis:Diode_DO-35, B.Cu at (235.6, 187.7)
- added KD24: 1N4148, travis:Diode_DO-35, B.Cu at (234.5, 149.6)
- added KD25: 1N4148, travis:Diode_DO-35, B.Cu at (233.3, 111.5)
- added KD26: 1N4148, travis:Diode_DO-35, B.Cu at (254.9, 188.3)
- added KD27: 1N4148, travis:Diode_DO-35, B.Cu at (254.4, 150.2)
- added KD28: 1N4148, travis:Diode_DO-35, B.Cu at (253.9, 112.1)
- added KD29: 1N4148, travis:Diode_DO-35, B.Cu at (274.1, 190.2)
- added KD3: 1N4148, travis:Diode_DO-35, B.Cu at (49.5, 115.3)
- added KD30: 1N4148, travis:Diode_DO-35, B.Cu at (274.2, 152.1)
- added KD31: 1N4148, travis:Diode_DO-35, B.Cu at (274.4, 114.0)
- added KD32: 1N4148, travis:Diode_DO-35, B.Cu at (293.1, 190.2)
- added KD33: 1N4148, travis:Diode_DO-35, B.Cu at (293.3, 152.1)
- added KD34: 1N4148, travis:Diode_DO-35, B.Cu at (293.5, 114.0)
- added KD35: 1N4148, travis:Diode_DO-35, B.Cu at (317.7, 152.2)
- added KD36: 1N4148, travis:Diode_DO-35, B.Cu at (312.5, 114.1)
- added KD37: 1N4148, travis:Diode_DO-35, B.Cu at (336.9, 114.2)
- added KD38: 1N4148, travis:Diode_DO-35, B.Cu at (336.9, 196.6)
- added KD39: 1N4148, travis:Diode_DO-35, B.Cu at (349.7, 182.4)
- added KD4: 1N4148, travis:Diode_DO-35, B.Cu at (69.2, 191.4)
- added KD40: 1N4148, travis:Diode_DO-35, B.Cu at (365.7, 164.8)
- added KD41: 1N4148, travis:Diode_DO-35, B.Cu at (378.5, 150.7)
- added KD42: 1N4148, travis:Diode_DO-35, B.Cu at (379.2, 114.4)
- added KD43: 1N4148, travis:Diode_DO-35, B.Cu at (398.2, 114.5)
- added KD44: 1N4148, travis:Diode_DO-35, B.Cu at (44.8, 172.5)
- added KD45: 1N4148, travis:Diode_DO-35, B.Cu at (44.4, 134.4)
- added KD46: 1N4148, travis:Diode_DO-35, B.Cu at (49.4, 96.3)
- added KD47: 1N4148, travis:Diode_DO-35, B.Cu at (69.1, 172.3)
- added KD48: 1N4148, travis:Diode_DO-35, B.Cu at (68.7, 134.2)
- added KD49: 1N4148, travis:Diode_DO-35, B.Cu at (88.6, 170.3)
- added KD5: 1N4148, travis:Diode_DO-35, B.Cu at (68.9, 153.3)
- added KD50: 1N4148, travis:Diode_DO-35, B.Cu at (88.9, 132.2)
- added KD51: 1N4148, travis:Diode_DO-35, B.Cu at (89.3, 94.1)
- added KD52: 1N4148, travis:Diode_DO-35, B.Cu at (108.1, 169.6)
- added KD53: 1N4148, travis:Diode_DO-35, B.Cu at (109.1, 131.5)
- added KD54: 1N4148, travis:Diode_DO-35, B.Cu at (110.1, 93.5)
- added KD55: 1N4148, travis:Diode_DO-35, B.Cu at (127.6, 171.3)
- added KD56: 1N4148, travis:Diode_DO-35, B.Cu at (129.3, 133.2)
- added KD57: 1N4148, travis:Diode_DO-35, B.Cu at (130.9, 95.2)
- added KD58: 1N4148, travis:Diode_DO-35, B.Cu at (146.7, 172.4)
- added KD59: 1N4148, travis:Diode_DO-35, B.Cu at (148.6, 134.4)
- added KD6: 1N4148, travis:Diode_DO-35, B.Cu at (68.6, 115.2)
- added KD60: 1N4148, travis:Diode_DO-35, B.Cu at (150.4, 96.3)
- added KD61: 1N4148, travis:Diode_DO-35, B.Cu at (196.6, 171.6)
- added KD62: 1N4148, travis:Diode_DO-35, B.Cu at (194.8, 133.5)
- added KD63: 1N4148, travis:Diode_DO-35, B.Cu at (192.9, 95.5)
- added KD64: 1N4148, travis:Diode_DO-35, B.Cu at (215.6, 170.4)
- added KD65: 1N4148, travis:Diode_DO-35, B.Cu at (213.8, 132.4)
- added KD66: 1N4148, travis:Diode_DO-35, B.Cu at (211.9, 94.3)
- added KD67: 1N4148, travis:Diode_DO-35, B.Cu at (235.1, 168.6)
- added KD68: 1N4148, travis:Diode_DO-35, B.Cu at (233.9, 130.6)
- added KD69: 1N4148, travis:Diode_DO-35, B.Cu at (232.7, 92.5)
- added KD7: 1N4148, travis:Diode_DO-35, B.Cu at (88.4, 189.4)
- added KD70: 1N4148, travis:Diode_DO-35, B.Cu at (254.6, 169.2)
- added KD71: 1N4148, travis:Diode_DO-35, B.Cu at (254.1, 131.1)
- added KD72: 1N4148, travis:Diode_DO-35, B.Cu at (253.6, 93.0)
- added KD73: 1N4148, travis:Diode_DO-35, B.Cu at (274.2, 171.1)
- added KD74: 1N4148, travis:Diode_DO-35, B.Cu at (274.3, 133.0)
- added KD75: 1N4148, travis:Diode_DO-35, B.Cu at (298.6, 171.2)
- added KD76: 1N4148, travis:Diode_DO-35, B.Cu at (293.4, 133.1)
- added KD77: 1N4148, travis:Diode_DO-35, B.Cu at (293.5, 95.0)
- added KD78: 1N4148, travis:Diode_DO-35, B.Cu at (312.4, 133.2)
- added KD79: 1N4148, travis:Diode_DO-35, B.Cu at (312.6, 95.1)
- added KD8: 1N4148, travis:Diode_DO-35, B.Cu at (88.8, 151.3)
- added KD80: 1N4148, travis:Diode_DO-35, B.Cu at (331.5, 133.3)
- added KD81: 1N4148, travis:Diode_DO-35, B.Cu at (331.6, 95.2)
- added KD82: 1N4148, travis:Diode_DO-35, B.Cu at (350.7, 95.2)
- added KD83: 1N4148, travis:Diode_DO-35, B.Cu at (322.8, 183.7)
- added KD84: 1N4148, travis:Diode_DO-35, B.Cu at (335.6, 169.6)
- added KD85: 1N4148, travis:Diode_DO-35, B.Cu at (351.6, 152.0)
- added KD86: 1N4148, travis:Diode_DO-35, B.Cu at (364.4, 137.9)
- added KD87: 1N4148, travis:Diode_DO-35, B.Cu at (379.3, 95.4)
- added KD88: 1N4148, travis:Diode_DO-35, B.Cu at (398.3, 95.4)
- added KD9: 1N4148, travis:Diode_DO-35, B.Cu at (89.1, 113.2)
- added KLED1: SK6812mini-e, travis:led_SK6812mini-e (per-key single-side), B.Cu at (41.8, 204.6)
- added KLED10: SK6812mini-e, travis:led_SK6812mini-e (per-key single-side), B.Cu at (98.8, 201.4)
- added KLED11: SK6812mini-e, travis:led_SK6812mini-e (per-key single-side), B.Cu at (99.8, 163.3)
- added KLED12: SK6812mini-e, travis:led_SK6812mini-e (per-key single-side), B.Cu at (100.7, 125.3)
- added KLED13: SK6812mini-e, travis:led_SK6812mini-e (per-key single-side), B.Cu at (119.3, 164.9)
- added KLED14: SK6812mini-e, travis:led_SK6812mini-e (per-key single-side), B.Cu at (121.0, 126.8)
- added KLED15: SK6812mini-e, travis:led_SK6812mini-e (per-key single-side), B.Cu at (135.2, 203.9)
- added KLED16: SK6812mini-e, travis:led_SK6812mini-e (per-key single-side), B.Cu at (138.5, 166.0)
- added KLED17: SK6812mini-e, travis:led_SK6812mini-e (per-key single-side), B.Cu at (140.3, 127.9)
- added KLED18: SK6812mini-e, travis:led_SK6812mini-e (per-key single-side), B.Cu at (191.1, 203.9)
- added KLED19: SK6812mini-e, travis:led_SK6812mini-e (per-key single-side), B.Cu at (187.8, 165.9)
- added KLED2: SK6812mini-e, travis:led_SK6812mini-e (per-key single-side), B.Cu at (36.2, 166.6)
- added KLED20: SK6812mini-e, travis:led_SK6812mini-e (per-key single-side), B.Cu at (186.0, 127.9)
- added KLED21: SK6812mini-e, travis:led_SK6812mini-e (per-key single-side), B.Cu at (206.8, 164.8)
- added KLED22: SK6812mini-e, travis:led_SK6812mini-e (per-key single-side), B.Cu at (205.0, 126.7)
- added KLED23: SK6812mini-e, travis:led_SK6812mini-e (per-key single-side), B.Cu at (227.5, 200.9)
- added KLED24: SK6812mini-e, travis:led_SK6812mini-e (per-key single-side), B.Cu at (226.4, 162.8)
- added KLED25: SK6812mini-e, travis:led_SK6812mini-e (per-key single-side), B.Cu at (225.2, 124.8)
- added KLED26: SK6812mini-e, travis:led_SK6812mini-e (per-key single-side), B.Cu at (246.5, 201.3)
- added KLED27: SK6812mini-e, travis:led_SK6812mini-e (per-key single-side), B.Cu at (246.0, 163.3)
- added KLED28: SK6812mini-e, travis:led_SK6812mini-e (per-key single-side), B.Cu at (245.5, 125.2)
- added KLED29: SK6812mini-e, travis:led_SK6812mini-e (per-key single-side), B.Cu at (265.5, 203.1)
- added KLED3: SK6812mini-e, travis:led_SK6812mini-e (per-key single-side), B.Cu at (41.1, 128.4)
- added KLED30: SK6812mini-e, travis:led_SK6812mini-e (per-key single-side), B.Cu at (265.7, 165.0)
- added KLED31: SK6812mini-e, travis:led_SK6812mini-e (per-key single-side), B.Cu at (265.8, 126.9)
- added KLED32: SK6812mini-e, travis:led_SK6812mini-e (per-key single-side), B.Cu at (284.5, 203.2)
- added KLED33: SK6812mini-e, travis:led_SK6812mini-e (per-key single-side), B.Cu at (284.7, 165.1)
- added KLED34: SK6812mini-e, travis:led_SK6812mini-e (per-key single-side), B.Cu at (284.9, 127.0)
- added KLED35: SK6812mini-e, travis:led_SK6812mini-e (per-key single-side), B.Cu at (309.1, 165.2)
- added KLED36: SK6812mini-e, travis:led_SK6812mini-e (per-key single-side), B.Cu at (303.9, 127.1)
- added KLED37: SK6812mini-e, travis:led_SK6812mini-e (per-key single-side), B.Cu at (328.3, 127.2)
- added KLED38: SK6812mini-e, travis:led_SK6812mini-e (per-key single-side), B.Cu at (340.8, 211.6)
- added KLED39: SK6812mini-e, travis:led_SK6812mini-e (per-key single-side), B.Cu at (353.6, 197.5)
- added KLED4: SK6812mini-e, travis:led_SK6812mini-e (per-key single-side), B.Cu at (60.8, 204.4)
- added KLED40: SK6812mini-e, travis:led_SK6812mini-e (per-key single-side), B.Cu at (369.6, 179.9)
- added KLED41: SK6812mini-e, travis:led_SK6812mini-e (per-key single-side), B.Cu at (382.4, 165.8)
- added KLED42: SK6812mini-e, travis:led_SK6812mini-e (per-key single-side), B.Cu at (370.6, 127.4)
- added KLED43: SK6812mini-e, travis:led_SK6812mini-e (per-key single-side), B.Cu at (389.6, 127.4)
- added KLED44: SK6812mini-e, travis:led_SK6812mini-e (per-key single-side), B.Cu at (36.4, 185.6)
- added KLED45: SK6812mini-e, travis:led_SK6812mini-e (per-key single-side), B.Cu at (36.0, 147.5)
- added KLED46: SK6812mini-e, travis:led_SK6812mini-e (per-key single-side), B.Cu at (41.0, 109.4)
- added KLED47: SK6812mini-e, travis:led_SK6812mini-e (per-key single-side), B.Cu at (60.7, 185.4)
- added KLED48: SK6812mini-e, travis:led_SK6812mini-e (per-key single-side), B.Cu at (60.3, 147.3)
- added KLED49: SK6812mini-e, travis:led_SK6812mini-e (per-key single-side), B.Cu at (79.9, 183.2)
- added KLED5: SK6812mini-e, travis:led_SK6812mini-e (per-key single-side), B.Cu at (60.5, 166.3)
- added KLED50: SK6812mini-e, travis:led_SK6812mini-e (per-key single-side), B.Cu at (80.3, 145.1)
- added KLED51: SK6812mini-e, travis:led_SK6812mini-e (per-key single-side), B.Cu at (80.6, 107.0)
- added KLED52: SK6812mini-e, travis:led_SK6812mini-e (per-key single-side), B.Cu at (99.3, 182.4)
- added KLED53: SK6812mini-e, travis:led_SK6812mini-e (per-key single-side), B.Cu at (100.2, 144.3)
- added KLED54: SK6812mini-e, travis:led_SK6812mini-e (per-key single-side), B.Cu at (101.2, 106.2)
- added KLED55: SK6812mini-e, travis:led_SK6812mini-e (per-key single-side), B.Cu at (118.5, 183.9)
- added KLED56: SK6812mini-e, travis:led_SK6812mini-e (per-key single-side), B.Cu at (120.2, 145.8)
- added KLED57: SK6812mini-e, travis:led_SK6812mini-e (per-key single-side), B.Cu at (121.8, 107.8)
- added KLED58: SK6812mini-e, travis:led_SK6812mini-e (per-key single-side), B.Cu at (137.6, 185.0)
- added KLED59: SK6812mini-e, travis:led_SK6812mini-e (per-key single-side), B.Cu at (139.4, 146.9)
- added KLED6: SK6812mini-e, travis:led_SK6812mini-e (per-key single-side), B.Cu at (60.2, 128.2)
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Other:
- board text added: "KC1"
- board text added: "KC10"
- board text added: "KC11"
- board text added: "KC12"
- board text added: "KC13"
- board text added: "KC14"
- board text added: "KC15"
- board text added: "KC16"
- board text added: "KC17"
- board text added: "KC18"
- board text added: "KC19"
- board text added: "KC2"
- board text added: "KC20"
- board text added: "KC21"
- board text added: "KC22"
- board text added: "KC23"
- board text added: "KC24"
- board text added: "KC25"
- board text added: "KC26"
- board text added: "KC27"
- board text added: "KC28"
- board text added: "KC29"
- board text added: "KC3"
- board text added: "KC30"
- board text added: "KC31"
- board text added: "KC32"
- board text added: "KC33"
- board text added: "KC34"
- board text added: "KC35"
- board text added: "KC36"
- board text added: "KC37"
- board text added: "KC38"
- board text added: "KC39"
- board text added: "KC4"
- board text added: "KC40"
- board text added: "KC41"
- board text added: "KC42"
- board text added: "KC43"
- board text added: "KC44"
- board text added: "KC45"
- board text added: "KC46"
- board text added: "KC47"
- board text added: "KC48"
- board text added: "KC49"
- board text added: "KC5"
- board text added: "KC50"
- board text added: "KC51"
- board text added: "KC52"
- board text added: "KC53"
- board text added: "KC54"
- board text added: "KC55"
- board text added: "KC56"
- board text added: "KC57"
- board text added: "KC58"
- board text added: "KC59"
- board text added: "KC6"
- board text added: "KC60"
- board text added: "KC61"
- board text added: "KC62"
- board text added: "KC63"
- board text added: "KC64"
- board text added: "KC65"
- board text added: "KC66"
- board text added: "KC67"
- board text added: "KC68"
- board text added: "KC69"
- board text added: "KC7"
- board text added: "KC70"
- board text added: "KC71"
- board text added: "KC72"
- board text added: "KC73"
- board text added: "KC74"
- board text added: "KC75"
- board text added: "KC76"
- board text added: "KC77"
- board text added: "KC78"
- board text added: "KC79"
- board text added: "KC8"
- board text added: "KC80"
- board text added: "KC81"
- board text added: "KC82"
- board text added: "KC83"
- board text added: "KC84"
- board text added: "KC85"
- board text added: "KC86"
- board text added: "KC87"
- board text added: "KC88"
- board text added: "KC9"
- board text added: "KD1"
- board text added: "KD10"
- board text added: "KD11"
- board text added: "KD12"
- board text added: "KD13"
- board text added: "KD14"
- board text added: "KD15"
- board text added: "KD16"
- board text added: "KD17"
- board text added: "KD18"
- board text added: "KD19"
- board text added: "KD2"
- board text added: "KD20"
- board text added: "KD21"
- board text added: "KD22"
- board text added: "KD23"
- board text added: "KD24"
- board text added: "KD25"
- board text added: "KD26"
- board text added: "KD27"
- board text added: "KD28"
- board text added: "KD29"
- board text added: "KD3"
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
Commit message: updating routes
Connections:
- DIP1 pad 10: row2 -> col0
- DIP1 pad 11: row3 -> col1
- DIP1 pad 12: row4 -> col2
- DIP1 pad 13: row5 -> col3
- DIP1 pad 14: col0 -> col4
- DIP1 pad 15: col1 -> col5
- MCU1 pad 10: col2 -> row5
- MCU1 pad 17: mux0 -> mux3
- MCU1 pad 18: mux1 -> mux2
- MCU1 pad 19: mux2 -> mux1
- MCU1 pad 20: mux3 -> mux0
- MCU1 pad 21: scrA -> scrC
- MCU1 pad 22: scrC -> scrA
- MCU1 pad 7: col5 -> row2
- MCU1 pad 8: col4 -> row3
- MCU1 pad 9: col3 -> row4
Other:
- board text added: "2024.03.25"
- board text removed: "2024.03.23"

Commit message: footprint/module updates
Parts:
- C1: footprint travis:C_Radial_D6.3mm_H11.0mm_P2.50mm -> Capacitor_THT:C_Radial_D6.3mm_H11.0mm_P2.50mm
- C2, C3: footprint travis:C_Disc_D3.8mm_W2.6mm_P2.50mm -> Capacitor_THT:C_Disc_D3.8mm_W2.6mm_P2.50mm
- D1, D2, KD1, KD10, KD11, KD12, KD13, KD14, KD15, KD16, KD17, KD18, KD19, KD2, KD20, KD21, KD22, KD23, KD24, KD25, KD26, KD27, KD28, KD29, KD3, KD30, KD31, KD32, KD33, KD34, KD35, KD36, KD37, KD38, KD39, KD4, KD40, KD41, KD42, KD43, KD44, KD45, KD46, KD47, KD48, KD49, KD5, KD50, KD51, KD52, KD53, KD54, KD55, KD56, KD57, KD58, KD59, KD6, KD60, KD61, KD62, KD63, KD64, KD65, KD66, KD67, KD68, KD69, KD7, KD70, KD71, KD72, KD73, KD74, KD75, KD76, KD77, KD78, KD79, KD8, KD80, KD81, KD82, KD83, KD84, KD85, KD86, KD87, KD88, KD9: footprint travis:Diode_DO-35 -> ScottoKeebs_Components:Diode_DO-35
- DIP1, DIP2: footprint travis:DIP-16_W7.62mm_Socket -> Package_DIP:DIP-16_W7.62mm_Socket
- KC1, KC10, KC11, KC12, KC13, KC14, KC15, KC16, KC17, KC18, KC19, KC2, KC20, KC21, KC22, KC23, KC24, KC25, KC26, KC27, KC28, KC29, KC3, KC30, KC31, KC32, KC33, KC34, KC35, KC36, KC37, KC38, KC39, KC4, KC40, KC41, KC42, KC43, KC44, KC45, KC46, KC47, KC48, KC49, KC5, KC50, KC51, KC52, KC53, KC54, KC55, KC56, KC57, KC58, KC59, KC6, KC60, KC61, KC62, KC63, KC64, KC65, KC66, KC67, KC68, KC69, KC7, KC70, KC71, KC72, KC73, KC74, KC75, KC76, KC77, KC78, KC79, KC8, KC80, KC81, KC82, KC83, KC84, KC85, KC86, KC87, KC88, KC9: footprint travis:C_Disc_D4.7mm_W2.5mm_P5.00mm -> Capacitor_THT:C_Disc_D4.7mm_W2.5mm_P5.00mm
- R1: footprint travis:R_Axial_DIN0207_L6.3mm_D2.5mm_P10.16mm_Horizontal -> Resistor_THT:R_Axial_DIN0207_L6.3mm_D2.5mm_P10.16mm_Horizontal
- STAB2u1, STAB2u2: footprint travis:Stabilizer_MX_2.00u -> ScottoKeebs_Stabilizer:Stabilizer_MX_2.00u
- SW1: footprint travis:SW_PUSH_6mm_H4.3mm -> Button_Switch_THT:SW_PUSH_6mm_H4.3mm
- SYM1: footprint travis:KiCad-Logo_5mm_Copper -> Symbol:KiCad-Logo_5mm_Copper
