File: key/output/pcbs/travis_key-ltr.kicad_pcb (KiCad board)
At the start: 2 copper layers, 38.1 x 38.1 mm, 4 parts

Commit message: footprint wip
Parts:
- LED1: value (none) -> SK6812mini-e; footprint ceoloide:led_SK6812mini-e (per-keysingle-side) -> ceoloide:led_SK6812mini-e (per-key single-side)
- moved D1 0.50 mm to (8.53, -8.03)
Connections:
- net LED_0 renamed LED_2
Routing:
- net single_A_one: track 5.29 -> 5.79 mm
Other:
- board text added: "C1"
- board text added: "D1"
- board text added: "LED_1"
